File: USB_UART_Converter.sch (KiCad schematic (older format))
At the start: 8 parts, among them J701 USB_B, U702 TPD3S014DBVR

Commit message: Updated UART USB converter sheet, and isolation sheet
Parts:
- removed D701: Green, LEDs:LED_0603, symbol Custom-Library:LED_ALT_Custom
- removed R703: 1k, Resistors_SMD:R_0603, symbol VFD_Clock-rescue:Res_Custom
- added C? (x2): 0.1uF, Capacitors_SMD:C_0603, symbol Custom-Library:C_Custom
- added C? (x2): 10nF, Capacitors_SMD:C_0603, symbol Custom-Library:C_Custom
- added C?: 4.7uF, Capacitors_SMD:C_0603, symbol Custom-Library:C_Custom
- added C? (x2): 47pF, Capacitors_SMD:C_0603, symbol Custom-Library:C_Custom
- added L?: 600R 0.5A, symbol Device:Ferrite_Bead
- added R? (x2): 27, Resistors_SMD:R_0603, symbol Device:R
- added R?: 10k, Resistors_SMD:R_0603, symbol VFD_Clock-rescue:Res_Custom
- added U?: FT234XD, Housings_DFN_QFN:DFN-12-1EP_3x3mm_Pitch0.45mm, symbol Custom_Library:FT234XD
Connections:
- net labels added: USB_DTR_ISO, ~USB_ACTIVE
- net labels removed: ~RXLED, ~TXLED
- wire segments 14 -> 43
- no-connect marks 1 -> 3
Other:
- note removed: "SWITCH TO FT234"

Commit message: Added a ton of test points and more indicators for system state
Parts:
- added TP?: TP, Measurement_Points:Measurement_Point_Round-SMD-Pad_Small, symbol Custom_Library:TP
- added TP?: TP, Pin_Headers:Pin_Header_Straight_1x01_Pitch2.54mm, symbol Custom_Library:TP
Connections:
- wire segments 43 -> 45
Changed lines of the file:
@@
 L Custom-Library:+5V_USB #PWR705
 U 1 1 5B3CEE8F
-P 6060 1980
-F 0 "#PWR705" H 6060 1830 50  0001 C CNN
-F 1 "+5V_USB" H 6060 2120 50  0000 C CNN
-F 2 "" H 6060 1980 50  0001 C CNN
-F 3 "" H 6060 1980 50  0001 C CNN
-	1    6060 1980
+P 5600 1940
+F 0 "#PWR705" H 5600 1790 50  0001 C CNN
+F 1 "+5V_USB" H 5600 2080 50  0000 C CNN
+F 2 "" H 5600 1940 50  0001 C CNN
+F 3 "" H 5600 1940 50  0001 C CNN
+	1    5600 1940
 	-1   0    0    1
 $EndComp
@@
 L power:PWR_FLAG #FLG701
 U 1 1 5B3CEF08
-P 6060 1980
-F 0 "#FLG701" H 6060 2055 50  0001 C CNN
-F 1 "PWR_FLAG" H 6060 2130 50  0000 C CNN
-F 2 "" H 6060 1980 50  0001 C CNN
-F 3 "" H 6060 1980 50  0001 C CNN
-	1    6060 1980
+P 5600 1940
+F 0 "#FLG701" H 5600 2015 50  0001 C CNN
+F 1 "PWR_FLAG" H 5600 2090 50  0000 C CNN
+F 2 "" H 5600 1940 50  0001 C CNN
+F 3 "" H 5600 1940 50  0001 C CNN
+	1    5600 1940
 	1    0    0    -1
 $EndComp
@@
 Wire Wire Line
 	1850 3480 2540 3480
+$Comp
+L Custom_Library:TP TP?
+U 1 1 5B532D6D
+P 6220 1990
+AR Path="/5A557C58/5B532D6D" Ref="TP?"  Part="1"
+AR Path="/5A0A8BD0/5B532D6D" Ref="TP?"  Part="1"
+F 0 "TP?" H 6220 2140 50  0000 C CNN
+F 1 "TP" H 6220 2140 50  0001 C CNN
+F 2 "Measurement_Points:Measurement_Point_Round-SMD-Pad_Small" H 6220 1990 60  0001 C CNN
+F 3 "" H 6220 1990 60  0000 C CNN
+	1    6220 1990
+	1    0    0    -1
+$EndComp
+Wire Wire Line
+	6220 1990 6220 2060
+Wire Wire Line
+	6220 2060 6600 2060
+$Comp
+L Custom_Library:TP TP?
+U 1 1 5B53630B
+P 8170 3950
+AR Path="/5A557C58/5B53630B" Ref="TP?"  Part="1"
+AR Path="/5A0A3EA5/5B53630B" Ref="TP?"  Part="1"
+F 0 "TP?" H 8170 4100 50  0000 C CNN
+F 1 "TP" H 8170 4100 50  0001 C CNN
+F 2 "Pin_Headers:Pin_Header_Straight_1x01_Pitch2.54mm" H 8170 3950 60  0001 C CNN
+F 3 "" H 8170 3950 60  0000 C CNN
+	1    8170 3950
+	1    0    0    -1
+$EndComp
+$Comp
+L Custom-Library:GND_USB #PWR?
+U 1 1 5B536CFC
+P 8170 3950
+F 0 "#PWR?" H 8170 3700 50  0001 C CNN
+F 1 "GND_USB" H 8170 3800 50  0000 C CNN
+F 2 "" H 8170 3950 50  0001 C CNN
+F 3 "" H 8170 3950 50  0001 C CNN
+	1    8170 3950
+	1    0    0    -1
+$EndComp
 $EndSCHEMATC

Commit message: Added a config field for every part, DNP some I2C pullups, added I2C header, changed some serial port functionality
Parts:
- added C?: 0.1uF, Capacitors_SMD:C_0603, symbol Custom-Library:C_Custom
- added U?: 74LVC1G17, symbol Custom_Library:74LVC1G17_Power
Connections:
- wire segments 45 -> 47
Changed lines of the file:
@@
 	1    0    0    -1
 $EndComp
-Text GLabel 1850 3480 0    60   Output ~ 0
+Text GLabel 1330 4790 0    60   Output ~ 0
 USB_DTR_ISO
-Wire Wire Line
-	1850 3480 2540 3480
 $Comp
 L Custom_Library:TP TP?
@@
 	1    0    0    -1
 $EndComp
+$Comp
+L Custom-Library:GND_USB #PWR?
+U 1 1 5B50A840
+P 1580 4890
+F 0 "#PWR?" H 1580 4640 50  0001 C CNN
+F 1 "GND_USB" H 1580 4740 50  0000 C CNN
+F 2 "" H 1580 4890 50  0001 C CNN
+F 3 "" H 1580 4890 50  0001 C CNN
+	1    1580 4890
+	1    0    0    -1
+$EndComp
+$Comp
+L Custom-Library:+5V_USB #PWR?
+U 1 1 5B50C4F8
+P 1580 4690
+F 0 "#PWR?" H 1580 4540 50  0001 C CNN
+F 1 "+5V_USB" H 1580 4840 50  0000 C CNN
+F 2 "" H 1580 4690 50  0001 C CNN
+F 3 "" H 1580 4690 50  0001 C CNN
+	1    1580 4690
+	1    0    0    -1
+$EndComp
+$Comp
+L Custom-Library:C_Custom C?
+U 1 1 5B50DE5A
+P 1420 5510
+F 0 "C?" H 1445 5610 50  0000 L CNN
+F 1 "0.1uF" H 1445 5410 50  0000 L CNN
+F 2 "Capacitors_SMD:C_0603" H 1458 5360 50  0001 C CNN
+F 3 "" H 1445 5610 50  0001 C CNN
+F 4 "0603" H 1270 5610 50  0000 R CNN "display_footprint"
+F 5 "50V" H 1270 5510 50  0000 R CNN "Voltage"
+F 6 "X7R" H 1270 5410 50  0000 R CNN "Dielectric"
+	1    1420 5510
+	1    0    0    -1
+$EndComp
+$Comp
+L Custom-Library:GND_USB #PWR?
+U 1 1 5B50DE61
+P 1420 5660
+F 0 "#PWR?" H 1420 5410 50  0001 C CNN
+F 1 "GND_USB" H 1420 5510 50  0000 C CNN
+F 2 "" H 1420 5660 50  0001 C CNN
+F 3 "" H 1420 5660 50  0001 C CNN
+	1    1420 5660
+	1    0    0    -1
+$EndComp
+$Comp
+L Custom-Library:+5V_USB #PWR?
+U 1 1 5B50DE67
+P 1420 5360
+F 0 "#PWR?" H 1420 5210 50  0001 C CNN
+F 1 "+5V_USB" H 1420 5500 50  0000 C CNN
+F 2 "" H 1420 5360 50  0001 C CNN
+F 3 "" H 1420 5360 50  0001 C CNN
+	1    1420 5360
+	1    0    0    -1
+$EndComp
+Wire Wire Line
+	1880 4790 2090 4790
+Wire Wire Line
+	2090 4790 2090 3480
+Wire Wire Line
+	2090 3480 2540 3480
+$Comp
+L Custom_Library:74LVC1G17_Power U?
+U 1 1 5B519C6A
+P 1580 4790
+F 0 "U?" H 1480 4940 50  0000 R CNN
+F 1 "74LVC1G17" H 1200 4660 50  0000 C CNN
+F 2 "" H 1580 4790 50  0001 C CNN
+F 3 "http://www.ti.com/lit/sg/scyt129e/scyt129e.pdf" H 1580 4790 50  0001 C CNN
+	1    1580 4790
+	-1   0    0    -1
+$EndComp
 $EndSCHEMATC

Commit message: Annotated all components, finished assigning footprints, netlist generated
Parts:
- L701: renamed from L?; footprint (none) -> Inductors_SMD:L_0603
- U701: renamed from U?; footprint (none) -> TO_SOT_Packages_SMD:SOT-363_SC-70-6; Digi-Key PN (none) -> 296-16998-1-ND
- gave numbers to parts that had none: 14
Connections:
- wire segments 47 -> 48

Commit message: Changed POS3P3 MOSFETs, further schematic enhancements, footprint updates, and arranged a few more pages of components on PCB
Parts:
- removed J701: USB_B, Connectors:USB_B, symbol Connector:USB_B
- added J701: USB_B_Micro, Connectors_USB:USB_Micro-B_Wuerth-629105150521_CircularHoles, symbol Connector:USB_B_Micro
Connections:
- no-connect marks 3 -> 4
Changed lines of the file:
@@
 	0    -1   -1   0
-$EndComp
-$Comp
-L Connector:USB_B J701
-U 1 1 5A1943A5
-P 9500 3180
-F 0 "J701" H 9300 3630 50  0000 L CNN
-F 1 "USB_B" H 9300 3530 50  0000 L CNN
-F 2 "Connectors:USB_B" H 9650 3130 50  0001 C CNN
-F 3 "" H 9650 3130 50  0001 C CNN
-	1    9500 3180
-	-1   0    0    -1
 $EndComp
 Wire Wire Line
@@
 	8680 1980 8680 2060
 Connection ~ 8680 2060
+$Comp
+L Connector:USB_B_Micro J701
+U 1 1 5B57F956
+P 9500 3180
+F 0 "J701" H 9300 3630 50  0000 L CNN
+F 1 "USB_B_Micro" H 9300 3530 50  0000 L CNN
+F 2 "Connectors_USB:USB_Micro-B_Wuerth-629105150521_CircularHoles" H 9650 3130 50  0001 C CNN
+F 3 "~" H 9650 3130 50  0001 C CNN
+F 4 "732-5960-1-ND" H 9500 3180 50  0001 C CNN "Digi-Key PN"
+	1    9500 3180
+	-1   0    0    -1
+$EndComp
+NoConn ~ 9200 3380
 $EndSCHEMATC
