File: BackupSupply.sch (KiCad schematic (older format))
At the start: 26 parts

Commit message: Resolved an issue with the field names of resistors on anode and grid driver sheets
Parts:
- C? (x2): display_foot TH -> (none); display_footprint (none) -> TH
Changed lines of the file:
@@
 F 2 "" H 4260 3430 50  0001 C CNN
 F 3 "" H 4285 3530 50  0001 C CNN
-F 4 "TH" H 4110 3330 50  0000 R CNN "display_foot"
+F 4 "TH" H 4110 3330 50  0000 R CNN "display_footprint"
 F 5 "V" H 4110 3530 50  0000 R CNN "Voltage"
 	1    4260 3430
@@
 F 2 "" H 4260 3990 50  0001 C CNN
 F 3 "" H 4285 4090 50  0001 C CNN
-F 4 "TH" H 4110 3890 50  0000 R CNN "display_foot"
+F 4 "TH" H 4110 3890 50  0000 R CNN "display_footprint"
 F 5 "V" H 4110 4090 50  0000 R CNN "Voltage"
 	1    4260 3990

Commit message: Changed the status sheet drastically to use I/O expander, and changed PGOOD sheet to include HOLDUP_PGOOD LED
Parts:
- added TP? (x2): TP, symbol Custom_Library:TP
Connections:
- net labels added: HOLDUP_PGOOD, VHU, ~HOLDUP_UV
- net labels removed: CAP_PGOOD, ~CAP_UV
- wire segments 98 -> 100
Changed lines of the file:
@@
 	2100 5050 1440 5050
 Text GLabel 1360 5050 0    60   Output ~ 0
-CAP_PGOOD
+HOLDUP_PGOOD
 Wire Wire Line
 	1360 5050 1440 5050
@@
 ~POS3P3_UV
 Text GLabel 8390 4310 2    60   Output ~ 0
-~CAP_UV
+~HOLDUP_UV
 Wire Wire Line
 	8390 4210 7610 4210
@@
 	8390 4310 8310 4310
 Connection ~ 8310 4310
+$Comp
+L Custom_Library:VHU #PWR?
+U 1 1 5B50B4E4
+P 4260 3070
+F 0 "#PWR?" H 4260 2920 50  0001 C CNN
+F 1 "VHU" H 4260 3220 50  0000 C CNN
+F 2 "" H 4260 3070 50  0001 C CNN
+F 3 "" H 4260 3070 50  0001 C CNN
+	1    4260 3070
+	1    0    0    -1
+$EndComp
+Wire Wire Line
+	4260 3070 4260 3150
+Text GLabel 9730 4420 3    60   Output ~ 0
+~HOLDUP_UV
+$Comp
+L Custom_Library:TP TP?
+U 1 1 5B51014B
+P 9730 4420
+F 0 "TP?" H 9730 4570 50  0000 C CNN
+F 1 "TP" H 9730 4570 50  0001 C CNN
+F 2 "" H 9730 4420 60  0000 C CNN
+F 3 "" H 9730 4420 60  0000 C CNN
+	1    9730 4420
+	1    0    0    -1
+$EndComp
+$Comp
+L Custom_Library:TP TP?
+U 1 1 5B51077B
+P 4960 3070
+F 0 "TP?" H 4960 3220 50  0000 C CNN
+F 1 "TP" H 4960 3220 50  0001 C CNN
+F 2 "" H 4960 3070 60  0000 C CNN
+F 3 "" H 4960 3070 60  0000 C CNN
+	1    4960 3070
+	1    0    0    -1
+$EndComp
+Wire Wire Line
+	4960 3070 4960 3150
 $EndSCHEMATC

Commit message: Added HOLDUP voltage ADC monitoring
Parts:
- added R?: 0, symbol Custom_Library:R_Custom
Connections:
- net labels added: HOLDUP_ADC
- wire segments 100 -> 103
Changed lines of the file:
@@
 $EndComp
 Wire Wire Line
-	5950 4510 4960 4510
+	5950 4510 5380 4510
 Connection ~ 4960 4510
 Wire Wire Line
@@
 Wire Wire Line
 	4960 3070 4960 3150
+$Comp
+L Custom_Library:R_Custom R?
+U 1 1 5B51C67B
+P 5630 5240
+F 0 "R?" V 5530 5240 50  0000 C CNN
+F 1 "0" V 5630 5240 50  0000 C CNN
+F 2 "" H 5630 5240 50  0001 C CNN
+F 3 "" H 5630 5240 50  0001 C CNN
+F 4 "0603" V 5730 5240 50  0000 C CNN "display_footprint"
+F 5 "1%" V 5830 5240 50  0000 C CNN "Tolerance"
+F 6 "1/10W" V 5930 5240 50  0000 C CNN "Wattage"
+F 7 "PN" H 5930 5640 60  0001 C CNN "Digi-Key PN"
+	1    5630 5240
+	0    1    1    0
+$EndComp
+Wire Wire Line
+	5480 5240 5380 5240
+Wire Wire Line
+	5380 5240 5380 4510
+Connection ~ 5380 4510
+Wire Wire Line
+	5380 4510 4960 4510
+Text GLabel 5780 5240 2    60   Output ~ 0
+HOLDUP_ADC
 $EndSCHEMATC

Commit message: Added a ton of test points and more indicators for system state
Parts:
- removed TP? (x2): TP, symbol Custom_Library:TP
- added TP? (x2): TP, Measurement_Points:Measurement_Point_Round-SMD-Pad_Small, symbol Custom_Library:TP
Changed lines of the file:
@@
 Wire Wire Line
 	4260 3070 4260 3150
-Text GLabel 9730 4420 3    60   Output ~ 0
-~HOLDUP_UV
-$Comp
-L Custom_Library:TP TP?
-U 1 1 5B51014B
-P 9730 4420
-F 0 "TP?" H 9730 4570 50  0000 C CNN
-F 1 "TP" H 9730 4570 50  0001 C CNN
-F 2 "" H 9730 4420 60  0000 C CNN
-F 3 "" H 9730 4420 60  0000 C CNN
-	1    9730 4420
-	1    0    0    -1
-$EndComp
-$Comp
-L Custom_Library:TP TP?
-U 1 1 5B51077B
-P 4960 3070
-F 0 "TP?" H 4960 3220 50  0000 C CNN
-F 1 "TP" H 4960 3220 50  0001 C CNN
-F 2 "" H 4960 3070 60  0000 C CNN
-F 3 "" H 4960 3070 60  0000 C CNN
-	1    4960 3070
-	1    0    0    -1
-$EndComp
 Wire Wire Line
 	4960 3070 4960 3150
@@
 Text GLabel 5780 5240 2    60   Output ~ 0
 HOLDUP_ADC
+$Comp
+L Custom_Library:TP TP?
+U 1 1 5B523282
+P 10140 1630
+F 0 "TP?" H 10140 1780 50  0000 C CNN
+F 1 "TP" H 10140 1780 50  0001 C CNN
+F 2 "Measurement_Points:Measurement_Point_Round-SMD-Pad_Small" H 10140 1630 60  0001 C CNN
+F 3 "" H 10140 1630 60  0000 C CNN
+	1    10140 1630
+	1    0    0    -1
+$EndComp
+$Comp
+L Custom-Library:+3.3V_MNG #PWR?
+U 1 1 5B5233DA
+P 10140 1630
+F 0 "#PWR?" H 10140 1480 50  0001 C CNN
+F 1 "+3.3V_MNG" H 10140 1770 50  0000 C CNN
+F 2 "" H 10140 1630 50  0000 C CNN
+F 3 "" H 10140 1630 50  0000 C CNN
+	1    10140 1630
+	-1   0    0    1
+$EndComp
+$Comp
+L Custom_Library:TP TP?
+U 1 1 5B523B1A
+P 4960 3070
+F 0 "TP?" H 4960 3220 50  0000 C CNN
+F 1 "TP" H 4960 3220 50  0001 C CNN
+F 2 "Measurement_Points:Measurement_Point_Round-SMD-Pad_Small" H 4960 3070 60  0001 C CNN
+F 3 "" H 4960 3070 60  0000 C CNN
+	1    4960 3070
+	1    0    0    -1
+$EndComp
 $EndSCHEMATC

Commit message: Found component values for holdup circuits
Parts:
- removed C?: C, symbol Custom-Library:CP1_Alum_Custom
- removed C? (x2): C, symbol Custom-Library:C_Custom
- added C?: 15F, symbol Custom-Library:CP1_Alum_Custom
- added C? (x2): 10uF, symbol Custom-Library:C_Custom
- C?: value C -> 15F; Digi-Key PN (none) -> 478-10017-ND; Voltage V -> 2.7V
- C?: value C_Custom -> 470pF; Dielectric Er -> X7R; Voltage V -> 50V; display_footprint Foot -> 0603
- C?: value C -> 10uF; Dielectric Er -> X7R; Voltage V -> 6.3V; display_footprint Foot -> 1206
- L?: value L_Custom -> 3.3uH; Ampacity A -> 5.5A; Digi-Key PN (none) -> 541-1237-1-ND; display_footprint Foot -> IHLP2020
- R?: value R -> 3.6k
- R?: value R -> 2.2M
- R?: value R -> 3.65k
- R?: value R -> 340k
- R?: value R -> 124k
- R?: value R -> 1M
- R?: value R -> 324k
- R?: value R -> 276k
Other:
- note added: "VHU = 4.3V\n~V1_UV~ => VHU = 2.31V\n~V2_UV~ => VHU = 2.89V\nSwitchover => +3.3V = 2.805V"
Changed lines of the file:
@@
 P 2950 2760
 F 0 "L?" V 2900 2760 50  0000 C CNN
-F 1 "L_Custom" V 3025 2760 50  0000 C CNN
+F 1 "3.3uH" V 3025 2760 50  0000 C CNN
 F 2 "" H 2950 2760 50  0001 C CNN
 F 3 "" H 2950 2760 50  0001 C CNN
-F 4 "Foot" V 3100 2760 50  0000 C CNN "display_footprint"
-F 5 "A" V 3200 2760 50  0000 C CNN "Ampacity"
+F 4 "IHLP2020" V 3100 2760 50  0000 C CNN "display_footprint"
+F 5 "5.5A" V 3200 2760 50  0000 C CNN "Ampacity"
 F 6 "Tol" V 3300 2760 50  0001 C CNN "Tolerance"
+F 7 "541-1237-1-ND" V 2950 2760 50  0001 C CNN "Digi-Key PN"
 	1    2950 2760
 	0    -1   -1   0
@@
 P 4260 3430
 F 0 "C?" H 4285 3530 50  0000 L CNN
-F 1 "C" H 4285 3330 50  0000 L CNN
+F 1 "15F" H 4285 3330 50  0000 L CNN
 F 2 "" H 4260 3430 50  0001 C CNN
 F 3 "" H 4285 3530 50  0001 C CNN
 F 4 "TH" H 4110 3330 50  0000 R CNN "display_footprint"
-F 5 "V" H 4110 3530 50  0000 R CNN "Voltage"
+F 5 "2.7V" H 4110 3530 50  0000 R CNN "Voltage"
+F 6 "478-10017-ND" H 4260 3430 50  0001 C CNN "Digi-Key PN"
 	1    4260 3430
-	1    0    0    -1
-$EndComp
-$Comp
-L Custom-Library:CP1_Alum_Custom C?
-U 1 1 5B4D1540
-P 4260 3990
-F 0 "C?" H 4285 4090 50  0000 L CNN
-F 1 "C" H 4285 3890 50  0000 L CNN
-F 2 "" H 4260 3990 50  0001 C CNN
-F 3 "" H 4285 4090 50  0001 C CNN
-F 4 "TH" H 4110 3890 50  0000 R CNN "display_footprint"
-F 5 "V" H 4110 4090 50  0000 R CNN "Voltage"
-	1    4260 3990
 	1    0    0    -1
 $EndComp
@@
 AR Path="/5A557C58/5B4D5A16" Ref="R?"  Part="1"
 F 0 "R?" H 4120 5580 50  0000 R CNN
-F 1 "R" V 4180 5580 50  0000 C CNN
+F 1 "3.6k" V 4180 5580 50  0000 C CNN
 F 2 "Resistors_SMD:R_0603" H 4180 5580 50  0001 C CNN
 F 3 "" H 4180 5580 50  0001 C CNN
@@
 L Custom-Library:C_Custom C?
 U 1 1 5B4D6BB1
-P 4740 5610
-F 0 "C?" H 4765 5710 50  0000 L CNN
-F 1 "C_Custom" H 4765 5510 50  0000 L CNN
-F 2 "" H 4778 5460 50  0001 C CNN
-F 3 "" H 4765 5710 50  0001 C CNN
-F 4 "Foot" H 4590 5710 50  0000 R CNN "display_footprint"
-F 5 "V" H 4590 5610 50  0000 R CNN "Voltage"
-F 6 "Er" H 4590 5510 50  0000 R CNN "Dielectric"
-F 7 "PN" H 5165 6110 60  0001 C CNN "Digi-Key PN"
-	1    4740 5610
+P 4880 5610
+F 0 "C?" H 4905 5710 50  0000 L CNN
+F 1 "470pF" H 4905 5510 50  0000 L CNN
+F 2 "" H 4918 5460 50  0001 C CNN
+F 3 "" H 4905 5710 50  0001 C CNN
+F 4 "0603" H 4730 5710 50  0000 R CNN "display_footprint"
+F 5 "50V" H 4730 5610 50  0000 R CNN "Voltage"
+F 6 "X7R" H 4730 5510 50  0000 R CNN "Dielectric"
+F 7 "PN" H 5305 6110 60  0001 C CNN "Digi-Key PN"
+	1    4880 5610
 	1    0    0    -1
 $EndComp
@@
 L power:GND #PWR?
 U 1 1 5B4D6C22
-P 4740 5760
-F 0 "#PWR?" H 4740 5510 50  0001 C CNN
-F 1 "GND" H 4740 5610 50  0000 C CNN
-F 2 "" H 4740 5760 50  0001 C CNN
-F 3 "" H 4740 5760 50  0001 C CNN
-	1    4740 5760
-	1    0    0    -1
-$EndComp
-Wire Wire Line
-	4740 5460 4740 5350
-Wire Wire Line
-	4740 5350 4180 5350
+P 4880 5760
+F 0 "#PWR?" H 4880 5510 50  0001 C CNN
+F 1 "GND" H 4880 5610 50  0000 C CNN
+F 2 "" H 4880 5760 50  0001 C CNN
+F 3 "" H 4880 5760 50  0001 C CNN
+	1    4880 5760
+	1    0    0    -1
+$EndComp
+Wire Wire Line
+	4880 5460 4880 5350
+Wire Wire Line
+	4880 5350 4180 5350
 Connection ~ 4180 5350
 $Comp
@@
 AR Path="/5A557C58/5B4D784A" Ref="R?"  Part="1"
 F 0 "R?" H 4900 3880 50  0000 R CNN
-F 1 "R" V 4960 3880 50  0000 C CNN
+F 1 "2.2M" V 4960 3880 40  0000 C CNN
 F 2 "Resistors_SMD:R_0603" H 4960 3880 50  0001 C CNN
 F 3 "" H 4960 3880 50  0001 C CNN
@@
 AR Path="/5A557C58/5B4D78AB" Ref="R?"  Part="1"
 F 0 "R?" H 4900 4280 50  0000 R CNN
-F 1 "R" V 4960 4280 50  0000 C CNN
+F 1 "3.65k" V 4960 4280 40  0000 C CNN
 F 2 "Resistors_SMD:R_0603" H 4960 4280 50  0001 C CNN
 F 3 "" H 4960 4280 50  0001 C CNN
@@
 AR Path="/5A557C58/5B4D78FB" Ref="R?"  Part="1"
 F 0 "R?" H 4900 4690 50  0000 R CNN
-F 1 "R" V 4960 4690 50  0000 C CNN
+F 1 "340k" V 4960 4690 40  0000 C CNN
 F 2 "Resistors_SMD:R_0603" H 4960 4690 50  0001 C CNN
 F 3 "" H 4960 4690 50  0001 C CNN
@@
 AR Path="/5A557C58/5B4DADC7" Ref="R?"  Part="1"
 F 0 "R?" H 2090 5870 50  0000 L CNN
-F 1 "R" V 2020 5710 50  0000 C CNN
+F 1 "124k" V 2020 5710 40  0000 C CNN
 F 2 "Resistors_SMD:R_0603" H 2020 5710 50  0001 C CNN
 F 3 "" H 2020 5710 50  0001 C CNN
@@
 $EndComp
 $Comp
-L Custom-Library:C_Custom C?
-U 1 1 5B51A9B3
-P 1490 3640
-F 0 "C?" H 1515 3740 50  0000 L CNN
-F 1 "C" H 1515 3540 50  0000 L CNN
-F 2 "" H 1528 3490 50  0001 C CNN
-F 3 "" H 1515 3740 50  0001 C CNN
-F 4 "Foot" H 1340 3740 50  0000 R CNN "display_footprint"
-F 5 "V" H 1340 3640 50  0000 R CNN "Voltage"
-F 6 "Er" H 1340 3540 50  0000 R CNN "Dielectric"
-F 7 "PN" H 1915 4140 60  0001 C CNN "Digi-Key PN"
-	1    1490 3640
-	1    0    0    -1
-$EndComp
-$Comp
 L power:GND #PWR?
 U 1 1 5B51AF9B
@@
 P 940 3640
 F 0 "C?" H 965 3740 50  0000 L CNN
-F 1 "C" H 965 3540 50  0000 L CNN
+F 1 "10uF" H 965 3540 50  0000 L CNN
 F 2 "" H 978 3490 50  0001 C CNN
 F 3 "" H 965 3740 50  0001 C CNN
-F 4 "Foot" H 790 3740 50  0000 R CNN "display_footprint"
-F 5 "V" H 790 3640 50  0000 R CNN "Voltage"
-F 6 "Er" H 790 3540 50  0000 R CNN "Dielectric"
+F 4 "1206" H 790 3740 50  0000 R CNN "display_footprint"
+F 5 "6.3V" H 790 3640 50  0000 R CNN "Voltage"
+F 6 "X7R" H 790 3540 50  0000 R CNN "Dielectric"
 F 7 "PN" H 1365 4140 60  0001 C CNN "Digi-Key PN"
 	1    940  3640
@@
 AR Path="/5A557C58/5B53AF32" Ref="R?"  Part="1"
 F 0 "R?" H 5650 2710 50  0000 R CNN
-F 1 "R" V 5710 2710 50  0000 C CNN
+F 1 "1M" V 5710 2710 50  0000 C CNN
 F 2 "Resistors_SMD:R_0603" H 5710 2710 50  0001 C CNN
 F 3 "" H 5710 2710 50  0001 C CNN
@@
 AR Path="/5A557C58/5B53AF3C" Ref="R?"  Part="1"
 F 0 "R?" H 5650 3180 50  0000 R CNN
-F 1 "R" V 5710 3180 50  0000 C CNN
+F 1 "324k" V 5710 3180 40  0000 C CNN
 F 2 "Resistors_SMD:R_0603" H 5710 3180 50  0001 C CNN
 F 3 "" H 5710 3180 50  0001 C CNN
@@
 AR Path="/5A557C58/5B53AF46" Ref="R?"  Part="1"
 F 0 "R?" H 5650 3590 50  0000 R CNN
-F 1 "R" V 5710 3590 50  0000 C CNN
+F 1 "276k" V 5710 3590 40  0000 C CNN
 F 2 "Resistors_SMD:R_0603" H 5710 3590 50  0001 C CNN
 F 3 "" H 5710 3590 50  0001 C CNN
@@
 Wire Wire Line
 	8310 4310 8310 4080
-$Comp
-L Custom-Library:C_Custom C?
-U 1 1 5B566F8E
-P 7350 2640
-F 0 "C?" H 7375 2740 50  0000 L CNN
-F 1 "C" H 7375 2540 50  0000 L CNN
-F 2 "" H 7388 2490 50  0001 C CNN
-F 3 "" H 7375 2740 50  0001 C CNN
-F 4 "Foot" H 7200 2740 50  0000 R CNN "display_footprint"
-F 5 "V" H 7200 2640 50  0000 R CNN "Voltage"
-F 6 "Er" H 7200 2540 50  0000 R CNN "Dielectric"
-F 7 "PN" H 7775 3140 60  0001 C CNN "Digi-Key PN"
-	1    7350 2640
-	1    0    0    -1
-$EndComp
 Wire Wire Line
 	7350 2490 7350 2410
@@
 	1    0    0    -1
 $EndComp
+$Comp
+L Custom-Library:CP1_Alum_Custom C?
+U 1 1 5B53BACE
+P 4260 3990
+F 0 "C?" H 4285 4090 50  0000 L CNN
+F 1 "15F" H 4285 3890 50  0000 L CNN
+F 2 "" H 4260 3990 50  0001 C CNN
+F 3 "" H 4285 4090 50  0001 C CNN
+F 4 "TH" H 4110 3890 50  0000 R CNN "display_footprint"
+F 5 "2.7V" H 4110 4090 50  0000 R CNN "Voltage"
+F 6 "478-10017-ND" H 4260 3990 50  0001 C CNN "Digi-Key PN"
+	1    4260 3990
+	1    0    0    -1
+$EndComp
+Text Notes 5020 1900 0    60   ~ 0
+VHU = 4.3V\n~V1_UV~ => VHU = 2.31V\n~V2_UV~ => VHU = 2.89V\nSwitchover => +3.3V = 2.805V
+$Comp
+L Custom-Library:C_Custom C?
+U 1 1 5B545555
+P 1490 3640
+F 0 "C?" H 1515 3740 50  0000 L CNN
+F 1 "10uF" H 1515 3540 50  0000 L CNN
+F 2 "" H 1528 3490 50  0001 C CNN
+F 3 "" H 1515 3740 50  0001 C CNN
+F 4 "1206" H 1340 3740 50  0000 R CNN "display_footprint"
+F 5 "6.3V" H 1340 3640 50  0000 R CNN "Voltage"
+F 6 "X7R" H 1340 3540 50  0000 R CNN "Dielectric"
+F 7 "PN" H 1915 4140 60  0001 C CNN "Digi-Key PN"
+	1    1490 3640
+	1    0    0    -1
+$EndComp
+$Comp
+L Custom-Library:C_Custom C?
+U 1 1 5B5467A5
+P 7350 2640
+F 0 "C?" H 7375 2740 50  0000 L CNN
+F 1 "10uF" H 7375 2540 50  0000 L CNN
+F 2 "" H 7388 2490 50  0001 C CNN
+F 3 "" H 7375 2740 50  0001 C CNN
+F 4 "1206" H 7200 2740 50  0000 R CNN "display_footprint"
+F 5 "6.3V" H 7200 2640 50  0000 R CNN "Voltage"
+F 6 "X7R" H 7200 2540 50  0000 R CNN "Dielectric"
+F 7 "PN" H 7775 3140 60  0001 C CNN "Digi-Key PN"
+	1    7350 2640
+	1    0    0    -1
+$EndComp

Commit message: Annotated all components, finished assigning footprints, netlist generated
Parts:
- C1701, C1702, C1706: renamed from C?; footprint (none) -> Capacitors_SMD:C_1206
- C1703, C1704: renamed from C?; footprint (none) -> Custom Footprints Library:SCCT30B156SRB
- C1705, C1708, C1709: renamed from C?; footprint (none) -> Capacitors_SMD:C_0603
- C1707: renamed from C?; footprint (none) -> Capacitors_SMD:C_0805
- L1701: renamed from L?; footprint (none) -> Inductors_SMD:L_Vishay_IHLP-2020
- R1708: renamed from R?; footprint (none) -> Resistors_SMD:R_0603
- gave numbers to parts that had none: 18
Connections:
- wire segments 103 -> 104

Commit message: Added a bunch of Digi-Key PN's
Parts:
- C1701, C1702, C1706: Digi-Key PN PN -> 399-4938-1-ND
- C1705: Digi-Key PN PN -> 399-1075-1-ND
- Q1701: Digi-Key PN (none) -> 2N7002-GMCCT-ND
- R1701, R1702, R1709, R1712, R1713: Digi-Key PN (none) -> 311-1.00MHRCT-ND
- R1703: Digi-Key PN (none) -> P124KHCT-ND
- R1704: Digi-Key PN (none) -> P3.60KHCT-ND
- R1705: Digi-Key PN (none) -> P2.20MHCT-ND
- R1706: Digi-Key PN (none) -> P3.65KHCT-ND
- R1707: Digi-Key PN (none) -> P340KHCT-ND
- R1708: Digi-Key PN PN -> P0.0GCT-ND
- R1710: Digi-Key PN (none) -> P324KHCT-ND
- R1711: Digi-Key PN (none) -> 541-267KHCT-ND
Changed lines of the file:
@@
 F 5 "1%" H 4250 5580 50  0000 L CNN "Tolerance"
 F 6 "1/10W" H 4250 5510 50  0000 L CNN "Wattage"
+F 7 "P3.60KHCT-ND" H 0   0   50  0001 C CNN "Digi-Key PN"
 	1    4180 5580
 	-1   0    0    1
@@
 F 5 "50V" H 4730 5610 50  0000 R CNN "Voltage"
 F 6 "X7R" H 4730 5510 50  0000 R CNN "Dielectric"
-F 7 "PN" H 5305 6110 60  0001 C CNN "Digi-Key PN"
+F 7 "399-1075-1-ND" H 5305 6110 60  0001 C CNN "Digi-Key PN"
 	1    4880 5610
 	1    0    0    -1
@@
 F 5 "1%" H 5030 3880 50  0000 L CNN "Tolerance"
 F 6 "1/10W" H 5030 3810 50  0000 L CNN "Wattage"
+F 7 "P2.20MHCT-ND" H 0   0   50  0001 C CNN "Digi-Key PN"
 	1    4960 3880
 	-1   0    0    1
@@
 F 5 "1%" H 5030 4280 50  0000 L CNN "Tolerance"
 F 6 "1/10W" H 5030 4210 50  0000 L CNN "Wattage"
+F 7 "P3.65KHCT-ND" H 0   0   50  0001 C CNN "Digi-Key PN"
 	1    4960 4280
 	-1   0    0    1
@@
 F 5 "1%" H 5030 4690 50  0000 L CNN "Tolerance"
 F 6 "1/10W" H 5030 4620 50  0000 L CNN "Wattage"
+F 7 "P340KHCT-ND" H 0   0   50  0001 C CNN "Digi-Key PN"
 	1    4960 4690
 	-1   0    0    1
@@
 F 5 "1%" H 2090 5710 50  0000 L CNN "Tolerance"
 F 6 "1/10W" H 2090 5640 50  0000 L CNN "Wattage"
+F 7 "P124KHCT-ND" H 0   0   50  0001 C CNN "Digi-Key PN"
 	1    2020 5710
 	1    0    0    1
@@
 F 5 "1%" H 1510 4500 50  0000 L CNN "Tolerance"
 F 6 "1/10W" H 1510 4430 50  0000 L CNN "Wattage"
+F 7 "311-1.00MHRCT-ND" H 0   0   50  0001 C CNN "Digi-Key PN"
 	1    1440 4500
 	-1   0    0    1
@@
 F 5 "1%" H 1920 3910 50  0000 L CNN "Tolerance"
 F 6 "1/10W" H 1920 3840 50  0000 L CNN "Wattage"
+F 7 "311-1.00MHRCT-ND" H 0   0   50  0001 C CNN "Digi-Key PN"
 	1    1850 3910
 	1    0    0    1
@@
 F 5 "6.3V" H 790 3640 50  0000 R CNN "Voltage"
 F 6 "X7R" H 790 3540 50  0000 R CNN "Dielectric"
-F 7 "PN" H 1365 4140 60  0001 C CNN "Digi-Key PN"
+F 7 "399-4938-1-ND" H 1365 4140 60  0001 C CNN "Digi-Key PN"
 	1    940  3640
 	1    0    0    -1
@@
 F 5 "1%" H 5780 2710 50  0000 L CNN "Tolerance"
 F 6 "1/10W" H 5780 2640 50  0000 L CNN "Wattage"
+F 7 "311-1.00MHRCT-ND" H 0   0   50  0001 C CNN "Digi-Key PN"
 	1    5710 2710
 	-1   0    0    1
@@
 F 5 "1%" H 5780 3180 50  0000 L CNN "Tolerance"
 F 6 "1/10W" H 5780 3110 50  0000 L CNN "Wattage"
+F 7 "P324KHCT-ND" H 0   0   50  0001 C CNN "Digi-Key PN"
 	1    5710 3180
 	-1   0    0    1
@@
 F 5 "1%" H 5780 3590 50  0000 L CNN "Tolerance"
 F 6 "1/10W" H 5780 3520 50  0000 L CNN "Wattage"
+F 7 "541-267KHCT-ND" H 0   0   50  0001 C CNN "Digi-Key PN"
 	1    5710 3590
 	-1   0    0    1
@@
 F 5 "1%" H 8380 3930 50  0000 L CNN "Tolerance"
 F 6 "1/10W" H 8380 3860 50  0000 L CNN "Wattage"
+F 7 "311-1.00MHRCT-ND" H 0   0   50  0001 C CNN "Digi-Key PN"
 	1    8310 3930
 	1    0    0    1
@@
 F 2 "TO_SOT_Packages_SMD:SOT-23" H 2150 6510 29  0001 C CNN
 F 3 "" H 1950 6410 60  0000 C CNN
+F 4 "2N7002-GMCCT-ND" H 0   0   50  0001 C CNN "Digi-Key PN"
 	1    1950 6410
 	-1   0    0    -1
@@
 F 5 "1%" V 5830 5240 50  0000 C CNN "Tolerance"
 F 6 "1/10W" V 5930 5240 50  0000 C CNN "Wattage"
-F 7 "PN" H 5930 5640 60  0001 C CNN "Digi-Key PN"
+F 7 "P0.0GCT-ND" H 5930 5640 60  0001 C CNN "Digi-Key PN"
 	1    5630 5240
 	0    1    1    0
@@
 F 5 "6.3V" H 1340 3640 50  0000 R CNN "Voltage"
 F 6 "X7R" H 1340 3540 50  0000 R CNN "Dielectric"
-F 7 "PN" H 1915 4140 60  0001 C CNN "Digi-Key PN"
+F 7 "399-4938-1-ND" H 1915 4140 60  0001 C CNN "Digi-Key PN"
 	1    1490 3640
 	1    0    0    -1
@@
 F 5 "6.3V" H 7200 2640 50  0000 R CNN "Voltage"
 F 6 "X7R" H 7200 2540 50  0000 R CNN "Dielectric"
-F 7 "PN" H 7775 3140 60  0001 C CNN "Digi-Key PN"
+F 7 "399-4938-1-ND" H 7775 3140 60  0001 C CNN "Digi-Key PN"
 	1    7350 2640
 	1    0    0    -1
@@
 F 5 "1%" H 7680 3930 50  0000 L CNN "Tolerance"
 F 6 "1/10W" H 7680 3860 50  0000 L CNN "Wattage"
+F 7 "311-1.00MHRCT-ND" H 0   0   50  0001 C CNN "Digi-Key PN"
 	1    7610 3930
 	1    0    0    1
