File: Tube_Life_Timer.sch (KiCad schematic (older format))
At the start: 9 parts

Commit message: Added a config field for every part, DNP some I2C pullups, added I2C header, changed some serial port functionality
Parts:
- R? (x2): Config (none) -> DNP
Changed lines of the file:
@@
 F 2 "Resistors_SMD:R_0603" H 7780 3870 50  0001 C CNN
 F 3 "" H 7780 3870 50  0001 C CNN
-F 4 "0603" H 7850 3950 50  0000 L CNN "display_footprint"
-F 5 "1%" H 7850 3870 50  0000 L CNN "Tolerance"
-F 6 "1/10W" H 7850 3800 50  0000 L CNN "Wattage"
+F 4 "DNP" H 7840 3730 50  0000 L CNN "Config"
+F 5 "0603" H 7850 3950 50  0000 L CNN "display_footprint"
+F 6 "1%" H 7850 3870 50  0000 L CNN "Tolerance"
+F 7 "1/10W" H 7850 3800 50  0000 L CNN "Wattage"
 	1    7780 3870
 	-1   0    0    1
@@
 F 2 "Resistors_SMD:R_0603" H 7230 3870 50  0001 C CNN
 F 3 "" H 7230 3870 50  0001 C CNN
-F 4 "0603" H 7300 3950 50  0000 L CNN "display_footprint"
-F 5 "1%" H 7300 3870 50  0000 L CNN "Tolerance"
-F 6 "1/10W" H 7300 3800 50  0000 L CNN "Wattage"
+F 4 "DNP" H 7300 3730 50  0000 L CNN "Config"
+F 5 "0603" H 7300 3950 50  0000 L CNN "display_footprint"
+F 6 "1%" H 7300 3870 50  0000 L CNN "Tolerance"
+F 7 "1/10W" H 7300 3800 50  0000 L CNN "Wattage"
 	1    7230 3870
 	-1   0    0    1

Commit message: Added I2C Address symbols for I2C devices
Parts:
- added A?: 0x6B, symbol Custom_Library:I2C_Address
Changed lines of the file:
@@
+	1    0    0    -1
+$EndComp
+$Comp
+L Custom_Library:I2C_Address A?
+U 1 1 5B59D543
+P 5530 4980
+F 0 "A?" H 5530 5230 60  0001 C CNN
+F 1 "0x6B" H 5080 4980 60  0000 L CNN
+F 2 "" H 5530 5330 60  0001 C CNN
+F 3 "" H 5530 5330 60  0001 C CNN
+	1    5530 4980
 	1    0    0    -1
 $EndComp

Commit message: Annotated all components, finished assigning footprints, netlist generated
Parts:
- A2201: renamed from A?; footprint (none) -> Oddities:Dummy_Empty
- U2201: renamed from U?; footprint (none) -> TO_SOT_Packages_SMD:SOT-353_SC-70-5; Digi-Key PN (none) -> 296-11602-1-ND
- gave numbers to parts that had none: 8
Changed lines of the file:
@@
 $EndDescr
 $Comp
-L Custom_Library:DS1683 U?
+L Custom_Library:DS1683 U2202
 U 1 1 5B5039F7
 P 5550 4100
-F 0 "U?" H 5550 3750 60  0000 C CNN
+F 0 "U2202" H 5550 3750 60  0000 C CNN
 F 1 "DS1683" H 5550 4450 60  0000 C CNN
 F 2 "Housings_SOIC:SOIC-8_3.9x4.9mm_Pitch1.27mm" H 5450 4400 60  0001 C CNN
@@
 NoConn ~ 5150 3900
 $Comp
-L power:GND #PWR?
+L power:GND #PWR02206
 U 1 1 5B50444E
 P 5070 4380
-F 0 "#PWR?" H 5070 4130 50  0001 C CNN
+F 0 "#PWR02206" H 5070 4130 50  0001 C CNN
 F 1 "GND" H 5070 4230 50  0000 C CNN
 F 2 "" H 5070 4380 50  0001 C CNN
@@
 	5070 4300 5150 4300
 $Comp
-L Custom_Library:+3.3V #PWR?
+L Custom_Library:+3.3V #PWR02209
 U 1 1 5B504491
 P 6030 3820
-F 0 "#PWR?" H 6030 3670 50  0001 C CNN
+F 0 "#PWR02209" H 6030 3670 50  0001 C CNN
 F 1 "+3.3V" H 6030 3960 50  0000 C CNN
 F 2 "" H 6030 3820 50  0000 C CNN
@@
 P 7230 3720
 AR Path="/5A0A42E8/5B5056BF" Ref="#PWR?"  Part="1"
-AR Path="/5B4B0915/5B5056BF" Ref="#PWR?"  Part="1"
-F 0 "#PWR?" H 7230 3570 50  0001 C CNN
+AR Path="/5B4B0915/5B5056BF" Ref="#PWR02210"  Part="1"
+F 0 "#PWR02210" H 7230 3570 50  0001 C CNN
 F 1 "+3.3V" H 7230 3860 50  0000 C CNN
 F 2 "" H 7230 3720 50  0001 C CNN
@@
 P 7780 3720
 AR Path="/5A0A42E8/5B5056C5" Ref="#PWR?"  Part="1"
-AR Path="/5B4B0915/5B5056C5" Ref="#PWR?"  Part="1"
-F 0 "#PWR?" H 7780 3570 50  0001 C CNN
+AR Path="/5B4B0915/5B5056C5" Ref="#PWR02211"  Part="1"
+F 0 "#PWR02211" H 7780 3570 50  0001 C CNN
 F 1 "+3.3V" H 7780 3860 50  0000 C CNN
 F 2 "" H 7780 3720 50  0001 C CNN
@@
 P 8190 4200
 AR Path="/5A0A42E8/5B5056D6" Ref="R?"  Part="1"
-AR Path="/5B4B0915/5B5056D6" Ref="R?"  Part="1"
-F 0 "R?" V 8090 4200 50  0000 C CNN
+AR Path="/5B4B0915/5B5056D6" Ref="R2204"  Part="1"
+F 0 "R2204" V 8090 4200 50  0000 C CNN
 F 1 "0" V 8190 4200 50  0000 C CNN
 F 2 "Resistors_SMD:R_0603" H 8190 4200 50  0001 C CNN
@@
 P 8190 4300
 AR Path="/5A0A42E8/5B5056E0" Ref="R?"  Part="1"
-AR Path="/5B4B0915/5B5056E0" Ref="R?"  Part="1"
-F 0 "R?" V 8090 4300 50  0000 C CNN
+AR Path="/5B4B0915/5B5056E0" Ref="R2205"  Part="1"
+F 0 "R2205" V 8090 4300 50  0000 C CNN
 F 1 "0" V 8180 4300 50  0000 C CNN
 F 2 "Resistors_SMD:R_0603" H 8190 4300 50  0001 C CNN
@@
 P 7780 3870
 AR Path="/5A0A42E8/5B5056EA" Ref="R?"  Part="1"
-AR Path="/5B4B0915/5B5056EA" Ref="R?"  Part="1"
-F 0 "R?" H 7720 3870 50  0000 R CNN
+AR Path="/5B4B0915/5B5056EA" Ref="R2203"  Part="1"
+F 0 "R2203" H 7720 3870 50  0000 R CNN
 F 1 "10k" V 7780 3870 50  0000 C CNN
 F 2 "Resistors_SMD:R_0603" H 7780 3870 50  0001 C CNN
@@
 P 7230 3870
 AR Path="/5A0A42E8/5B5056F4" Ref="R?"  Part="1"
-AR Path="/5B4B0915/5B5056F4" Ref="R?"  Part="1"
-F 0 "R?" H 7170 3870 50  0000 R CNN
+AR Path="/5B4B0915/5B5056F4" Ref="R2202"  Part="1"
+F 0 "R2202" H 7170 3870 50  0000 R CNN
 F 1 "10k" V 7230 3870 50  0000 C CNN
 F 2 "Resistors_SMD:R_0603" H 7230 3870 50  0001 C CNN
@@
 	7780 4300 5950 4300
 $Comp
-L Custom_Library:74LVC1G08_Power U?
+L Custom_Library:74LVC1G08_Power U2201
 U 1 1 5B505EF8
 P 3040 4100
-F 0 "U?" H 2940 4250 50  0000 R CNN
+F 0 "U2201" H 2940 4250 50  0000 R CNN
 F 1 "74LVC1G08" H 3350 3990 50  0000 C CNN
-F 2 "" H 3040 4100 50  0001 C CNN
+F 2 "TO_SOT_Packages_SMD:SOT-353_SC-70-5" H 3040 4100 50  0001 C CNN
 F 3 "http://www.ti.com/lit/sg/scyt129e/scyt129e.pdf" H 3040 4100 50  0001 C CNN
+F 4 "296-11602-1-ND" H 3040 4100 50  0001 C CNN "Digi-Key PN"
 	1    3040 4100
 	1    0    0    -1
 $EndComp
 $Comp
-L power:GND #PWR?
+L power:GND #PWR02204
 U 1 1 5B50648E
 P 3040 4200
-F 0 "#PWR?" H 3040 3950 50  0001 C CNN
+F 0 "#PWR02204" H 3040 3950 50  0001 C CNN
 F 1 "GND" H 3040 4050 50  0000 C CNN
 F 2 "" H 3040 4200 50  0001 C CNN
@@
 $EndComp
 $Comp
-L Custom_Library:+3.3V #PWR?
+L Custom_Library:+3.3V #PWR02203
 U 1 1 5B5064C1
 P 3040 4000
-F 0 "#PWR?" H 3040 3850 50  0001 C CNN
+F 0 "#PWR02203" H 3040 3850 50  0001 C CNN
 F 1 "+3.3V" H 3040 4140 50  0000 C CNN
 F 2 "" H 3040 4000 50  0000 C CNN
@@
 P 3900 4430
 AR Path="/5A0A42E8/5B506A12" Ref="R?"  Part="1"
-AR Path="/5B4B0915/5B506A12" Ref="R?"  Part="1"
-F 0 "R?" H 3840 4430 50  0000 R CNN
+AR Path="/5B4B0915/5B506A12" Ref="R2201"  Part="1"
+F 0 "R2201" H 3840 4430 50  0000 R CNN
 F 1 "10k" V 3900 4430 50  0000 C CNN
 F 2 "Resistors_SMD:R_0603" H 3900 4430 50  0001 C CNN
@@
 $EndComp
 $Comp
-L power:GND #PWR?
+L power:GND #PWR02205
 U 1 1 5B506A55
 P 3900 4580
-F 0 "#PWR?" H 3900 4330 50  0001 C CNN
+F 0 "#PWR02205" H 3900 4330 50  0001 C CNN
 F 1 "GND" H 3900 4430 50  0000 C CNN
 F 2 "" H 3900 4580 50  0001 C CNN
@@
 VFF_PGOOD
 $Comp
-L Custom-Library:C_Custom C?
+L Custom-Library:C_Custom C2202
 U 1 1 5B507AC7
 P 5540 3120
-F 0 "C?" H 5565 3220 50  0000 L CNN
+F 0 "C2202" H 5565 3220 50  0000 L CNN
 F 1 "0.1uF" H 5565 3020 50  0000 L CNN
 F 2 "Capacitors_SMD:C_0603" H 5578 2970 50  0001 C CNN
@@
 $EndComp
 $Comp
-L Custom_Library:+3.3V #PWR?
+L Custom_Library:+3.3V #PWR02207
 U 1 1 5B507B7D
 P 5540 2970
-F 0 "#PWR?" H 5540 2820 50  0001 C CNN
+F 0 "#PWR02207" H 5540 2820 50  0001 C CNN
 F 1 "+3.3V" H 5540 3110 50  0000 C CNN
 F 2 "" H 5540 2970 50  0000 C CNN
@@
 $EndComp
 $Comp
-L power:GND #PWR?
+L power:GND #PWR02208
 U 1 1 5B507BED
 P 5540 3270
-F 0 "#PWR?" H 5540 3020 50  0001 C CNN
+F 0 "#PWR02208" H 5540 3020 50  0001 C CNN
 F 1 "GND" H 5540 3120 50  0000 C CNN
 F 2 "" H 5540 3270 50  0001 C CNN
@@
 $EndComp
 $Comp
-L Custom-Library:C_Custom C?
+L Custom-Library:C_Custom C2201
 U 1 1 5B507D27
 P 2990 4890
-F 0 "C?" H 3015 4990 50  0000 L CNN
+F 0 "C2201" H 3015 4990 50  0000 L CNN
 F 1 "0.1uF" H 3015 4790 50  0000 L CNN
 F 2 "Capacitors_SMD:C_0603" H 3028 4740 50  0001 C CNN
@@
 $EndComp
 $Comp
-L Custom_Library:+3.3V #PWR?
+L Custom_Library:+3.3V #PWR02201
 U 1 1 5B507D2E
 P 2990 4740
-F 0 "#PWR?" H 2990 4590 50  0001 C CNN
+F 0 "#PWR02201" H 2990 4590 50  0001 C CNN
 F 1 "+3.3V" H 2990 4880 50  0000 C CNN
 F 2 "" H 2990 4740 50  0000 C CNN
@@
 $EndComp
 $Comp
-L power:GND #PWR?
+L power:GND #PWR02202
 U 1 1 5B507D34
 P 2990 5040
-F 0 "#PWR?" H 2990 4790 50  0001 C CNN
+F 0 "#PWR02202" H 2990 4790 50  0001 C CNN
 F 1 "GND" H 2990 4890 50  0000 C CNN
 F 2 "" H 2990 5040 50  0001 C CNN
@@
 $EndComp
 $Comp
-L Custom_Library:I2C_Address A?
+L Custom_Library:I2C_Address A2201
 U 1 1 5B59D543
 P 5530 4980
-F 0 "A?" H 5530 5230 60  0001 C CNN
+F 0 "A2201" H 5530 5230 60  0001 C CNN
 F 1 "0x6B" H 5080 4980 60  0000 L CNN
-F 2 "" H 5530 5330 60  0001 C CNN
+F 2 "Oddities:Dummy_Empty" H 5530 5330 60  0001 C CNN
 F 3 "" H 5530 5330 60  0001 C CNN
 	1    5530 4980

Commit message: Added a bunch of Digi-Key PN's
Parts:
- C2201, C2202: Digi-Key PN (none) -> 399-6856-1-ND
- R2201, R2202, R2203: Digi-Key PN (none) -> 541-10.0KHCT-ND
Changed lines of the file:
@@
 F 6 "1%" H 7850 3870 50  0000 L CNN "Tolerance"
 F 7 "1/10W" H 7850 3800 50  0000 L CNN "Wattage"
+F 8 "541-10.0KHCT-ND" H 0   0   50  0001 C CNN "Digi-Key PN"
 	1    7780 3870
 	-1   0    0    1
@@
 F 6 "1%" H 7300 3870 50  0000 L CNN "Tolerance"
 F 7 "1/10W" H 7300 3800 50  0000 L CNN "Wattage"
+F 8 "541-10.0KHCT-ND" H 0   0   50  0001 C CNN "Digi-Key PN"
 	1    7230 3870
 	-1   0    0    1
@@
 F 5 "1%" H 3970 4430 50  0000 L CNN "Tolerance"
 F 6 "1/10W" H 3970 4360 50  0000 L CNN "Wattage"
+F 7 "541-10.0KHCT-ND" H 0   0   50  0001 C CNN "Digi-Key PN"
 	1    3900 4430
 	-1   0    0    1
@@
 F 5 "50V" H 5390 3120 50  0000 R CNN "Voltage"
 F 6 "X7R" H 5390 3020 50  0000 R CNN "Dielectric"
+F 7 "399-6856-1-ND" H 0   0   50  0001 C CNN "Digi-Key PN"
 	1    5540 3120
 	1    0    0    -1
@@
 F 5 "50V" H 2840 4890 50  0000 R CNN "Voltage"
 F 6 "X7R" H 2840 4790 50  0000 R CNN "Dielectric"
+F 7 "399-6856-1-ND" H 0   0   50  0001 C CNN "Digi-Key PN"
 	1    2990 4890
 	1    0    0    -1

Commit message: Added slight logic changes to tube life timer sheet
Parts:
- added C2203: 0.1uF, Capacitors_SMD:C_0603, symbol Custom-Library:C_Custom
- added C2204, C2205, C2206: 10uF, Capacitors_SMD:C_1206, symbol Custom-Library:C_Custom
- added D2201: 1N5819, Diodes_SMD:D_SOD-123F, symbol Diode:1N5819
- added R2206: 10k, Resistors_SMD:R_0603, symbol Custom-Library:R_Custom
- added U2203: 74LVC1G38, TO_SOT_Packages_SMD:SOT-353_SC-70-5, symbol Custom-Library:74LVC1G38_Custom
Connections:
- wire segments 13 -> 30

Commit message: Finished POS3P3 redesign and cleaned other pages
Connections:
- wire segments 30 -> 31
Changed lines of the file:
@@
 	4760 4100 5150 4100
 Connection ~ 4760 4100
+$Comp
+L power:PWR_FLAG #FLG0105
+U 1 1 5B635A57
+P 6960 3820
+F 0 "#FLG0105" H 6960 3895 50  0001 C CNN
+F 1 "PWR_FLAG" H 6960 3970 50  0000 C CNN
+F 2 "" H 6960 3820 50  0001 C CNN
+F 3 "~" H 6960 3820 50  0001 C CNN
+	1    6960 3820
+	1    0    0    -1
+$EndComp
+Wire Wire Line
+	6960 3820 6960 3900
 $EndSCHEMATC

Commit message: Arranged more components on PCB, cleaned up schematic, added page titles, finished finding DigiKey PN's
Parts:
- R2201, R2206: Digi-Key PN 541-10.0KHCT-ND -> P10.0KHCT-ND
- R2204, R2205: Digi-Key PN (none) -> P0.0GCT-ND; Wattage 1/16W -> 1/10W; display_footprint 0402 -> 0603
Other:
- note added: "Tube Life Timer"
- moved on the sheet: D2201
