File: Microcontroller.sch (KiCad schematic (older format))
At the start: 21 parts, among them U301 PIC18LF67K40-I/PT, Y301 32.768kHz, Y302 16MHz

Commit message: Annotated all components, finished assigning footprints, netlist generated
Parts:
- A301: renamed from A?; footprint (none) -> Oddities:Dummy_Empty
- TP301: renamed from TP?; footprint (none) -> Pin_Headers:Pin_Header_Straight_1x03_Pitch2.54mm
- gave numbers to parts that had none: 1
Connections:
- net labels added: ~POS3P3_UV
- no-connect marks 0 -> 1
Changed lines of the file:
@@
 $EndDescr
 $Comp
-L power:GND #PWR308
+L power:GND #PWR0308
 U 1 1 5A49B2FB
 P 4750 7190
-F 0 "#PWR308" H 4750 6940 50  0001 C CNN
+F 0 "#PWR0308" H 4750 6940 50  0001 C CNN
 F 1 "GND" H 4750 7040 50  0000 C CNN
 F 2 "" H 4750 7190 50  0000 C CNN
@@
 $EndComp
 $Comp
-L power:GND #PWR315
+L power:GND #PWR0315
 U 1 1 5A49D84A
 P 9860 6100
-F 0 "#PWR315" H 9860 5850 50  0001 C CNN
+F 0 "#PWR0315" H 9860 5850 50  0001 C CNN
 F 1 "GND" H 9860 5950 50  0000 C CNN
 F 2 "" H 9860 6100 50  0001 C CNN
@@
 $EndComp
 $Comp
-L power:GND #PWR314
+L power:GND #PWR0314
 U 1 1 5A49D889
 P 9160 6100
-F 0 "#PWR314" H 9160 5850 50  0001 C CNN
+F 0 "#PWR0314" H 9160 5850 50  0001 C CNN
 F 1 "GND" H 9160 5950 50  0000 C CNN
 F 2 "" H 9160 6100 50  0001 C CNN
@@
 USB_DTR
 $Comp
-L VFD_Clock-rescue:+3.3V-RESCUE-VFD_Clock #PWR304
+L VFD_Clock-rescue:+3.3V-RESCUE-VFD_Clock #PWR0304
 U 1 1 5A4BF609
 P 2480 4150
-F 0 "#PWR304" H 2480 4000 50  0001 C CNN
+F 0 "#PWR0304" H 2480 4000 50  0001 C CNN
 F 1 "+3.3V" H 2480 4290 50  0000 C CNN
 F 2 "" H 2480 4150 50  0001 C CNN
@@
 $EndComp
 $Comp
-L VFD_Clock-rescue:+3.3V-RESCUE-VFD_Clock #PWR303
+L VFD_Clock-rescue:+3.3V-RESCUE-VFD_Clock #PWR0303
 U 1 1 5A4BF60F
 P 1930 4150
-F 0 "#PWR303" H 1930 4000 50  0001 C CNN
+F 0 "#PWR0303" H 1930 4000 50  0001 C CNN
 F 1 "+3.3V" H 1930 4290 50  0000 C CNN
 F 2 "" H 1930 4150 50  0001 C CNN
@@
 uC_OSC2
 $Comp
-L power:GND #PWR310
+L power:GND #PWR0310
 U 1 1 5A4D9A45
 P 5010 4960
-F 0 "#PWR310" H 5010 4710 50  0001 C CNN
+F 0 "#PWR0310" H 5010 4710 50  0001 C CNN
 F 1 "GND" H 5010 4810 50  0000 C CNN
 F 2 "" H 5010 4960 50  0001 C CNN
@@
 Connection ~ 5010 940
 $Comp
-L power:GND #PWR302
+L power:GND #PWR0302
 U 1 1 5A4E0653
 P 1620 7190
-F 0 "#PWR302" H 1620 6940 50  0001 C CNN
+F 0 "#PWR0302" H 1620 6940 50  0001 C CNN
 F 1 "GND" H 1620 7040 50  0000 C CNN
 F 2 "" H 1620 7190 50  0001 C CNN
@@
 $EndComp
 $Comp
-L power:GND #PWR313
+L power:GND #PWR0313
 U 1 1 5A55A471
 P 8130 6100
-F 0 "#PWR313" H 8130 5850 50  0001 C CNN
+F 0 "#PWR0313" H 8130 5850 50  0001 C CNN
 F 1 "GND" H 8130 5950 50  0000 C CNN
 F 2 "" H 8130 6100 50  0001 C CNN
@@
 $EndComp
 $Comp
-L power:GND #PWR312
+L power:GND #PWR0312
 U 1 1 5A55A477
 P 7430 6100
-F 0 "#PWR312" H 7430 5850 50  0001 C CNN
+F 0 "#PWR0312" H 7430 5850 50  0001 C CNN
 F 1 "GND" H 7430 5950 50  0000 C CNN
 F 2 "" H 7430 6100 50  0001 C CNN
@@
 uC_SOSC2
 $Comp
-L Custom-Library:+3.3V_MNG #PWR309
+L Custom-Library:+3.3V_MNG #PWR0309
 U 1 1 5A55ED44
 P 5010 900
-F 0 "#PWR309" H 5010 750 50  0001 C CNN
+F 0 "#PWR0309" H 5010 750 50  0001 C CNN
 F 1 "+3.3V_MNG" H 5010 1040 50  0000 C CNN
 F 2 "" H 5010 900 50  0000 C CNN
@@
 $EndComp
 $Comp
-L Custom-Library:+3.3V_MNG #PWR307
+L Custom-Library:+3.3V_MNG #PWR0307
 U 1 1 5A55F38D
 P 4750 6730
-F 0 "#PWR307" H 4750 6580 50  0001 C CNN
+F 0 "#PWR0307" H 4750 6580 50  0001 C CNN
 F 1 "+3.3V_MNG" H 4750 6870 50  0000 C CNN
 F 2 "" H 4750 6730 50  0000 C CNN
@@
 $EndComp
 $Comp
-L Custom-Library:+3.3V_MNG #PWR311
+L Custom-Library:+3.3V_MNG #PWR0311
 U 1 1 5A55F458
 P 5690 6860
-F 0 "#PWR311" H 5690 6710 50  0001 C CNN
+F 0 "#PWR0311" H 5690 6710 50  0001 C CNN
 F 1 "+3.3V_MNG" H 5690 7000 50  0000 C CNN
 F 2 "" H 5690 6860 50  0000 C CNN
@@
 $EndComp
 $Comp
-L Custom-Library:+3.3V_MNG #PWR301
+L Custom-Library:+3.3V_MNG #PWR0301
 U 1 1 5A55F493
 P 1620 6890
-F 0 "#PWR301" H 1620 6740 50  0001 C CNN
+F 0 "#PWR0301" H 1620 6740 50  0001 C CNN
 F 1 "+3.3V_MNG" H 1620 7030 50  0000 C CNN
 F 2 "" H 1620 6890 50  0000 C CNN
@@
 $EndComp
 $Comp
-L power:GND #PWR306
+L power:GND #PWR0306
 U 1 1 5AEE8EC0
 P 3230 7190
-F 0 "#PWR306" H 3230 6940 50  0001 C CNN
+F 0 "#PWR0306" H 3230 6940 50  0001 C CNN
 F 1 "GND" H 3230 7040 50  0000 C CNN
 F 2 "" H 3230 7190 50  0000 C CNN
@@
 $EndComp
 $Comp
-L Custom-Library:+3.3V_MNG #PWR305
+L Custom-Library:+3.3V_MNG #PWR0305
 U 1 1 5AEE8EEB
 P 3230 6730
-F 0 "#PWR305" H 3230 6580 50  0001 C CNN
+F 0 "#PWR0305" H 3230 6580 50  0001 C CNN
 F 1 "+3.3V_MNG" H 3230 6870 50  0000 C CNN
 F 2 "" H 3230 6730 50  0000 C CNN
@@
 Colon_2
 $Comp
-L Custom-Library:C_Custom C?
+L Custom-Library:C_Custom C301
 U 1 1 5B4EE115
 P 1620 7040
-F 0 "C?" H 1645 7140 50  0000 L CNN
+F 0 "C301" H 1645 7140 50  0000 L CNN
 F 1 "47uF" H 1645 6940 50  0000 L CNN
 F 2 "Capacitors_SMD:C_1210" H 1658 6890 50  0001 C CNN
@@
 HOLDUP_ADC
 $Comp
-L Connector_Generic:Conn_01x03 TP?
+L Connector_Generic:Conn_01x03 TP301
 U 1 1 5B5039B1
 P 1930 5460
-F 0 "TP?" H 1930 5660 50  0000 C CNN
+F 0 "TP301" H 1930 5660 50  0000 C CNN
 F 1 "I2C" H 1930 5260 50  0000 C CNN
-F 2 "" H 1930 5460 50  0001 C CNN
+F 2 "Pin_Headers:Pin_Header_Straight_1x03_Pitch2.54mm" H 1930 5460 50  0001 C CNN
 F 3 "~" H 1930 5460 50  0001 C CNN
 	1    1930 5460
@@
 $EndComp
 $Comp
-L power:GND #PWR?
+L power:GND #PWR0316
 U 1 1 5B504108
 P 1730 5560
-F 0 "#PWR?" H 1730 5310 50  0001 C CNN
+F 0 "#PWR0316" H 1730 5310 50  0001 C CNN
 F 1 "GND" H 1730 5410 50  0000 C CNN
 F 2 "" H 1730 5560 50  0001 C CNN
@@
 Encoder_STEP
 $Comp
-L Custom_Library:I2C_Address A?
+L Custom_Library:I2C_Address A301
 U 1 1 5B5967AF
 P 5010 5460
-F 0 "A?" H 5010 5710 60  0001 C CNN
+F 0 "A301" H 5010 5710 60  0001 C CNN
 F 1 "MASTER" H 4560 5460 60  0000 L CNN
-F 2 "" H 5010 5810 60  0001 C CNN
+F 2 "Oddities:Dummy_Empty" H 5010 5810 60  0001 C CNN
 F 3 "" H 5010 5810 60  0001 C CNN
 	1    5010 5460
 	1    0    0    -1
 $EndComp
+NoConn ~ 3760 3730
+Text GLabel 3760 3630 0    40   Input ~ 0
+~POS3P3_UV
 $EndSCHEMATC

Commit message: Switched to QFN micro, various footprint fixes, layed a a few more sheets out, changed puchbutton debouncers
Parts:
- removed U301: PIC18LF67K40-I/PT, Housings_QFP:TQFP-64_10x10mm_Pitch0.5mm, symbol VFD_Clock-rescue:PIC18(L)F67K40-I_PT
- added U301: PIC18LF67K40-I_MR, Housings_DFN_QFN:QFN-64-1EP_9x9mm_Pitch0.5mm, symbol Custom_Library:PIC18(L)F67K40-I_MR
Connections:
- wire segments 52 -> 53
Changed lines of the file:
@@
 Text GLabel 3760 1430 0    60   Input ~ 0
 POS24_CS_ADC
-Wire Wire Line
-	5010 4960 5010 4920
-Wire Wire Line
-	4960 4920 5010 4920
-Wire Wire Line
-	5060 4920 5060 4880
-Wire Wire Line
-	4960 4920 4960 4880
-Connection ~ 5010 4920
 Text GLabel 6260 4030 2    60   Output ~ 0
 Buzzer
@@
 Wire Wire Line
 	3230 7150 3230 7190
-Wire Wire Line
-	5010 4920 5060 4920
-$Comp
-L VFD_Clock-rescue:PIC18(L)F67K40-I_PT U301
-U 1 1 5B3C23A0
-P 5010 2980
-AR Path="/5B3C23A0" Ref="U301"  Part="1"
-AR Path="/5A0A42E8/5B3C23A0" Ref="U301"  Part="1"
-F 0 "U301" H 6060 1180 50  0000 R CNN
-F 1 "PIC18LF67K40-I/PT" H 5010 3030 50  0000 C CNN
-F 2 "Housings_QFP:TQFP-64_10x10mm_Pitch0.5mm" H 5010 5080 50  0001 C CNN
-F 3 "" H 4360 3630 50  0001 C CNN
-	1    5010 2980
-	1    0    0    -1
-$EndComp
 Text GLabel 6260 4130 2    60   Output ~ 0
 Colon_1
@@
 Text GLabel 3760 3630 0    40   Input ~ 0
 ~POS3P3_UV
+$Comp
+L Custom_Library:PIC18(L)F67K40-I_MR U301
+U 1 1 5B5806FA
+P 5010 2980
+F 0 "U301" H 6060 1180 50  0000 R CNN
+F 1 "PIC18LF67K40-I_MR" H 5010 3030 50  0000 C CNN
+F 2 "Housings_DFN_QFN:QFN-64-1EP_9x9mm_Pitch0.5mm" H 5010 5080 50  0001 C CNN
+F 3 "" H 4360 3630 50  0001 C CNN
+F 4 "PIC18LF67K40T-I/MRCT-ND" H 5010 2980 50  0001 C CNN "Digi-Key PN"
+	1    5010 2980
+	1    0    0    -1
+$EndComp
+Wire Wire Line
+	5010 4960 5010 4920
+Wire Wire Line
+	5010 4920 5110 4920
+Wire Wire Line
+	5110 4920 5110 4880
+Connection ~ 5010 4920
+Wire Wire Line
+	5010 4920 5010 4880
+Wire Wire Line
+	5010 4920 4910 4920
+Wire Wire Line
+	4910 4920 4910 4880
 $EndSCHEMATC

Commit message: Added a bunch of Digi-Key PN's
Parts:
- removed C301: 47uF, Capacitors_SMD:C_1210, symbol Custom-Library:C_Custom
- removed C310, C311: 18pF, Capacitors_SMD:C_0603, symbol Custom-Library:C_Custom
- removed Y302: 16MHz, Crystals:Crystal_SMD_SeikoEpson_FA238-4pin_3.2x2.5mm, symbol Device:Crystal
- C302, C305: Digi-Key PN (none) -> 399-6856-1-ND
- C303, C306: Digi-Key PN (none) -> 399-1092-1-ND
- C304, C307: Digi-Key PN (none) -> 399-1083-1-ND
- C308, C309: Digi-Key PN (none) -> 445-5046-1-ND
- R303, R304, R305: Digi-Key PN (none) -> 541-10.0KHCT-ND
Connections:
- net labels removed: uC_OSC1, uC_OSC2
- wire segments 53 -> 47
Other:
- note removed: "4X PLL -> FOSC = 64MHz"
- note removed: "Bulk"
Changed lines of the file:
@@
 F 5 "50V" H 4280 6960 50  0000 R CNN "Voltage"
 F 6 "X7R" H 4280 6860 50  0000 R CNN "Dielectric"
+F 7 "399-6856-1-ND" H 0   0   50  0001 C CNN "Digi-Key PN"
 	1    4430 6960
 	1    0    0    -1
@@
 F 5 "50V" H 4920 6960 50  0001 R CNN "Voltage"
 F 6 "X7R" H 4920 6860 50  0001 R CNN "Dielectric"
+F 7 "399-1083-1-ND" H 0   0   50  0001 C CNN "Digi-Key PN"
 	1    5070 6960
 	1    0    0    -1
@@
 F 5 "50V" H 4600 6960 50  0001 R CNN "Voltage"
 F 6 "X7R" H 4600 6860 50  0001 R CNN "Dielectric"
+F 7 "399-1092-1-ND" H 0   0   50  0001 C CNN "Digi-Key PN"
 	1    4750 6960
 	1    0    0    -1
@@
 F 5 "1%" H 5760 7010 50  0000 L CNN "Tolerance"
 F 6 "1/10W" H 5760 6940 50  0000 L CNN "Wattage"
+F 7 "541-10.0KHCT-ND" H 0   0   50  0001 C CNN "Digi-Key PN"
 	1    5690 7010
 	-1   0    0    1
@@
 Text GLabel 5690 7160 3    60   UnSpc ~ 0
 ~MCLR
-Text GLabel 9860 5520 1    60   UnSpc ~ 0
-uC_OSC2
-Text GLabel 9160 5520 1    60   UnSpc ~ 0
-uC_OSC1
-$Comp
-L Custom-Library:C_Custom C310
-U 1 1 5A49CF0D
-P 9160 5950
-F 0 "C310" H 9185 6050 50  0000 L CNN
-F 1 "18pF" H 9185 5850 50  0000 L CNN
-F 2 "Capacitors_SMD:C_0603" H 9198 5800 50  0001 C CNN
-F 3 "" H 9185 6050 50  0001 C CNN
-F 4 "0603" H 9010 6050 50  0000 R CNN "display_footprint"
-F 5 "50V" H 9010 5950 50  0000 R CNN "Voltage"
-F 6 "NP0" H 9010 5850 50  0000 R CNN "Dielectric"
-	1    9160 5950
-	1    0    0    -1
-$EndComp
-$Comp
-L Device:Crystal Y302
-U 1 1 5A49D355
-P 9510 5600
-F 0 "Y302" H 9510 5750 50  0000 C CNN
-F 1 "16MHz" H 9510 5450 50  0000 C CNN
-F 2 "Crystals:Crystal_SMD_SeikoEpson_FA238-4pin_3.2x2.5mm" H 9510 5600 50  0001 C CNN
-F 3 "" H 9510 5600 50  0001 C CNN
-F 4 "SER3686CT-ND" H 9510 5600 60  0001 C CNN "Digi-Key PN"
-	1    9510 5600
-	1    0    0    1
-$EndComp
-$Comp
-L Custom-Library:C_Custom C311
-U 1 1 5A49D3FB
-P 9860 5950
-F 0 "C311" H 9885 6050 50  0000 L CNN
-F 1 "18pF" H 9885 5850 50  0000 L CNN
-F 2 "Capacitors_SMD:C_0603" H 9898 5800 50  0001 C CNN
-F 3 "" H 9885 6050 50  0001 C CNN
-F 4 "0603" H 9710 6050 50  0000 R CNN "display_footprint"
-F 5 "50V" H 9710 5950 50  0000 R CNN "Voltage"
-F 6 "NP0" H 9710 5850 50  0000 R CNN "Dielectric"
-	1    9860 5950
-	-1   0    0    -1
-$EndComp
-$Comp
-L power:GND #PWR0315
-U 1 1 5A49D84A
-P 9860 6100
-F 0 "#PWR0315" H 9860 5850 50  0001 C CNN
-F 1 "GND" H 9860 5950 50  0000 C CNN
-F 2 "" H 9860 6100 50  0001 C CNN
-F 3 "" H 9860 6100 50  0001 C CNN
-	1    9860 6100
-	1    0    0    -1
-$EndComp
-$Comp
-L power:GND #PWR0314
-U 1 1 5A49D889
-P 9160 6100
-F 0 "#PWR0314" H 9160 5850 50  0001 C CNN
-F 1 "GND" H 9160 5950 50  0000 C CNN
-F 2 "" H 9160 6100 50  0001 C CNN
-F 3 "" H 9160 6100 50  0001 C CNN
-	1    9160 6100
-	1    0    0    -1
-$EndComp
-Wire Wire Line
-	9160 5520 9160 5600
-Wire Wire Line
-	9160 5600 9360 5600
-Wire Wire Line
-	9660 5600 9860 5600
-Wire Wire Line
-	9860 5520 9860 5600
-Connection ~ 9160 5600
-Connection ~ 9860 5600
-Text Notes 8800 4970 0    60   ~ 0
-4X PLL -> FOSC = 64MHz
 Text GLabel 6260 2130 2    60   Output ~ 0
 drive_Anode_A
@@
 F 5 "1%" H 2000 4300 50  0000 L CNN "Tolerance"
 F 6 "1/10W" H 2000 4230 50  0000 L CNN "Wattage"
+F 7 "541-10.0KHCT-ND" H 0   0   50  0001 C CNN "Digi-Key PN"
 	1    1930 4300
 	1    0    0    1
@@
 F 5 "1%" H 2550 4300 50  0000 L CNN "Tolerance"
 F 6 "1/10W" H 2550 4230 50  0000 L CNN "Wattage"
+F 7 "541-10.0KHCT-ND" H 0   0   50  0001 C CNN "Digi-Key PN"
 	1    2480 4300
 	1    0    0    1
@@
 Text GLabel 3760 1330 0    60   Input ~ 0
 POS24_ADC
-Text GLabel 3760 1930 0    60   UnSpc ~ 0
-uC_OSC1
-Text GLabel 3760 1830 0    60   UnSpc ~ 0
-uC_OSC2
 $Comp
 L power:GND #PWR0310
@@
 	5060 940  5060 980
 Connection ~ 5010 940
-$Comp
-L power:GND #PWR0302
-U 1 1 5A4E0653
-P 1620 7190
-F 0 "#PWR0302" H 1620 6940 50  0001 C CNN
-F 1 "GND" H 1620 7040 50  0000 C CNN
-F 2 "" H 1620 7190 50  0001 C CNN
-F 3 "" H 1620 7190 50  0001 C CNN
-	1    1620 7190
-	1    0    0    -1
-$EndComp
-Text Notes 1900 7030 0    60   ~ 0
-Bulk
 Text GLabel 6260 1430 2    40   Input ~ 0
 ~Time
@@
 F 5 "50V" H 7280 5950 50  0000 R CNN "Voltage"
 F 6 "NP0" H 7280 5850 50  0000 R CNN "Dielectric"
+F 7 "445-5046-1-ND" H 0   0   50  0001 C CNN "Digi-Key PN"
 	1    7430 5950
 	1    0    0    -1
@@
 F 5 "50V" H 7980 5950 50  0000 R CNN "Voltage"
 F 6 "NP0" H 7980 5850 50  0000 R CNN "Dielectric"
+F 7 "445-5046-1-ND" H 0   0   50  0001 C CNN "Digi-Key PN"
 	1    8130 5950
 	-1   0    0    -1
@@
 F 3 "" H 5690 6860 50  0000 C CNN
 	1    5690 6860
-	1    0    0    -1
-$EndComp
-$Comp
-L Custom-Library:+3.3V_MNG #PWR0301
-U 1 1 5A55F493
-P 1620 6890
-F 0 "#PWR0301" H 1620 6740 50  0001 C CNN
-F 1 "+3.3V_MNG" H 1620 7030 50  0000 C CNN
-F 2 "" H 1620 6890 50  0000 C CNN
-F 3 "" H 1620 6890 50  0000 C CNN
-	1    1620 6890
 	1    0    0    -1
 $EndComp
@@
 F 5 "50V" H 2760 6960 50  0000 R CNN "Voltage"
 F 6 "X7R" H 2760 6860 50  0000 R CNN "Dielectric"
+F 7 "399-6856-1-ND" H 0   0   50  0001 C CNN "Digi-Key PN"
 	1    2910 6960
 	1    0    0    -1
@@
 F 5 "50V" H 3400 6960 50  0001 R CNN "Voltage"
 F 6 "X7R" H 3400 6860 50  0001 R CNN "Dielectric"
+F 7 "399-1083-1-ND" H 0   0   50  0001 C CNN "Digi-Key PN"
 	1    3550 6960
 	1    0    0    -1
@@
 F 5 "50V" H 3080 6960 50  0001 R CNN "Voltage"
 F 6 "X7R" H 3080 6860 50  0001 R CNN "Dielectric"
+F 7 "399-1092-1-ND" H 0   0   50  0001 C CNN "Digi-Key PN"
 	1    3230 6960
 	1    0    0    -1
@@
 	4750 7150 4750 7190
 Wire Wire Line
-	9160 5600 9160 5800
-Wire Wire Line
-	9860 5600 9860 5800
-Wire Wire Line
 	2480 4530 3760 4530
 Wire Wire Line
@@
 Text GLabel 6260 4230 2    60   Output ~ 0
 Colon_2
-$Comp
-L Custom-Library:C_Custom C301
-U 1 1 5B4EE115
-P 1620 7040
-F 0 "C301" H 1645 7140 50  0000 L CNN
-F 1 "47uF" H 1645 6940 50  0000 L CNN
-F 2 "Capacitors_SMD:C_1210" H 1658 6890 50  0001 C CNN
-F 3 "" H 1645 7140 50  0001 C CNN
-F 4 "1210" H 1470 7140 50  0000 R CNN "display_footprint"
-F 5 "16V" H 1470 7040 50  0000 R CNN "Voltage"
-F 6 "X7R" H 1470 6940 50  0000 R CNN "Dielectric"
-	1    1620 7040
-	1    0    0    -1
-$EndComp
 Text GLabel 3760 3330 0    40   UnSpc ~ 0
 ~Status_Heartbeat

Commit message: Added input energy monitor
Connections:
- net labels added: ACCUM, REF_CLK
- no-connect marks 1 -> 0
Changed lines of the file:
@@
 	1    0    0    -1
 $EndComp
-Text GLabel 3760 3230 0    40   UnSpc ~ 0
+Text GLabel 3760 1830 0    40   UnSpc ~ 0
 ~Status_COM_Error
 Text GLabel 3760 1430 0    60   Input ~ 0
@@
 Text GLabel 6260 4230 2    60   Output ~ 0
 Colon_2
-Text GLabel 3760 3330 0    40   UnSpc ~ 0
+Text GLabel 3760 1930 0    40   UnSpc ~ 0
 ~Status_Heartbeat
-Text GLabel 3760 3430 0    60   Input ~ 0
+Text GLabel 3760 3230 0    60   Input ~ 0
 HOLDUP_PGOOD
 Text GLabel 6260 1330 2    60   Input ~ 0
 POS3P3_ADC
-Text GLabel 3760 3530 0    60   Input ~ 0
+Text GLabel 3760 3330 0    60   Input ~ 0
 HOLDUP_ADC
 $Comp
@@
 	1    0    0    -1
 $EndComp
-NoConn ~ 3760 3730
-Text GLabel 3760 3630 0    40   Input ~ 0
+Text GLabel 3760 3430 0    40   Input ~ 0
 ~POS3P3_UV
-$Comp
-L Custom_Library:PIC18(L)F67K40-I_MR U301
-U 1 1 5B5806FA
-P 5010 2980
-F 0 "U301" H 6060 1180 50  0000 R CNN
-F 1 "PIC18LF67K40-I_MR" H 5010 3030 50  0000 C CNN
-F 2 "Housings_DFN_QFN:QFN-64-1EP_9x9mm_Pitch0.5mm" H 5010 5080 50  0001 C CNN
-F 3 "" H 4360 3630 50  0001 C CNN
-F 4 "PIC18LF67K40T-I/MRCT-ND" H 5010 2980 50  0001 C CNN "Digi-Key PN"
-	1    5010 2980
-	1    0    0    -1
-$EndComp
 Wire Wire Line
 	5010 4960 5010 4920
@@
 Wire Wire Line
 	4910 4920 4910 4880
+Text GLabel 3760 3530 0    60   Output ~ 0
+ACCUM
+$Comp
+L Custom_Library:PIC18(L)F67K40-I_MR U301
+U 1 1 5B5806FA
+P 5010 2980
+F 0 "U301" H 6060 1180 50  0000 R CNN
+F 1 "PIC18LF67K40-I_MR" H 5010 3030 50  0000 C CNN
+F 2 "Housings_DFN_QFN:QFN-64-1EP_9x9mm_Pitch0.5mm" H 5010 5080 50  0001 C CNN
+F 3 "" H 4360 3630 50  0001 C CNN
+F 4 "PIC18LF67K40T-I/MRCT-ND" H 5010 2980 50  0001 C CNN "Digi-Key PN"
+	1    5010 2980
+	1    0    0    -1
+$EndComp
+Text GLabel 3760 3630 0    60   Output ~ 0
+REF_CLK
 $EndSCHEMATC

Commit message: Finished POS3P3 redesign and cleaned other pages
Connections:
- net labels removed: POS24_CS_ADC
Changed lines of the file:
@@
 Text GLabel 3760 1830 0    40   UnSpc ~ 0
 ~Status_COM_Error
-Text GLabel 3760 1430 0    60   Input ~ 0
-POS24_CS_ADC
 Text GLabel 6260 4030 2    60   Output ~ 0
 Buzzer

Commit message: Arranged more components on PCB, cleaned up schematic, added page titles, finished finding DigiKey PN's
Parts:
- added TP302: USB_UART, Pin_Headers:Pin_Header_Straight_1x03_Pitch2.54mm, symbol Connector_Generic:Conn_01x03
- R301, R302: Digi-Key PN (none) -> P0.0GCT-ND; Wattage 1/16W -> 1/10W; display_footprint 0402 -> 0603
- R303, R304, R305: Digi-Key PN 541-10.0KHCT-ND -> P10.0KHCT-ND
Connections:
- no-connect marks 0 -> 2
Other:
- note added: "8 Bit High Performance Microcontroller"
Changed lines of the file:
@@
 F 5 "1%" H 5760 7010 50  0000 L CNN "Tolerance"
 F 6 "1/10W" H 5760 6940 50  0000 L CNN "Wattage"
-F 7 "541-10.0KHCT-ND" H 0   0   50  0001 C CNN "Digi-Key PN"
+F 7 "P10.0KHCT-ND" H 0   0   50  0001 C CNN "Digi-Key PN"
 	1    5690 7010
 	-1   0    0    1
@@
 F 2 "Resistors_SMD:R_0603" H 1520 4530 50  0001 C CNN
 F 3 "" H 1520 4530 50  0001 C CNN
-F 4 "0402" V 1620 4530 50  0001 C CNN "display_footprint"
+F 4 "0603" V 1620 4530 50  0001 C CNN "display_footprint"
 F 5 "1%" V 1720 4530 50  0001 C CNN "Tolerance"
-F 6 "1/16W" V 1820 4530 50  0001 C CNN "Wattage"
+F 6 "1/10W" V 1820 4530 50  0001 C CNN "Wattage"
+F 7 "P0.0GCT-ND" H 0   0   50  0001 C CNN "Digi-Key PN"
 	1    1520 4530
 	0    -1   1    0
@@
 F 2 "Resistors_SMD:R_0603" H 1520 4630 50  0001 C CNN
 F 3 "" H 1520 4630 50  0001 C CNN
-F 4 "0402" V 1620 4630 50  0001 C CNN "display_footprint"
+F 4 "0603" V 1620 4630 50  0001 C CNN "display_footprint"
 F 5 "1%" V 1720 4630 50  0001 C CNN "Tolerance"
-F 6 "1/16W" V 1820 4630 50  0001 C CNN "Wattage"
+F 6 "1/10W" V 1820 4630 50  0001 C CNN "Wattage"
+F 7 "P0.0GCT-ND" H 0   0   50  0001 C CNN "Digi-Key PN"
 	1    1520 4630
 	0    -1   -1   0
@@
 F 5 "1%" H 2000 4300 50  0000 L CNN "Tolerance"
 F 6 "1/10W" H 2000 4230 50  0000 L CNN "Wattage"
-F 7 "541-10.0KHCT-ND" H 0   0   50  0001 C CNN "Digi-Key PN"
+F 7 "P10.0KHCT-ND" H 0   0   50  0001 C CNN "Digi-Key PN"
 	1    1930 4300
 	1    0    0    1
@@
 F 5 "1%" H 2550 4300 50  0000 L CNN "Tolerance"
 F 6 "1/10W" H 2550 4230 50  0000 L CNN "Wattage"
-F 7 "541-10.0KHCT-ND" H 0   0   50  0001 C CNN "Digi-Key PN"
+F 7 "P10.0KHCT-ND" H 0   0   50  0001 C CNN "Digi-Key PN"
 	1    2480 4300
 	1    0    0    1
@@
 Text GLabel 3760 3630 0    60   Output ~ 0
 REF_CLK
+NoConn ~ 3760 1430
+NoConn ~ 3760 3730
+$Comp
+L Connector_Generic:Conn_01x03 TP302
+U 1 1 5B5F52C3
+P 3430 5460
+F 0 "TP302" H 3430 5660 50  0000 C CNN
+F 1 "USB_UART" H 3430 5260 50  0000 L CNN
+F 2 "Pin_Headers:Pin_Header_Straight_1x03_Pitch2.54mm" H 3430 5460 50  0001 C CNN
+F 3 "~" H 3430 5460 50  0001 C CNN
+	1    3430 5460
+	1    0    0    -1
+$EndComp
+$Comp
+L power:GND #PWR0301
+U 1 1 5B5F52CA
+P 3230 5560
+F 0 "#PWR0301" H 3230 5310 50  0001 C CNN
+F 1 "GND" H 3230 5410 50  0000 C CNN
+F 2 "" H 3230 5560 50  0001 C CNN
+F 3 "" H 3230 5560 50  0001 C CNN
+	1    3230 5560
+	1    0    0    -1
+$EndComp
+Text GLabel 3230 5460 0    60   UnSpc ~ 0
+USB_UART_TX
+Text GLabel 3230 5360 0    60   UnSpc ~ 0
+USB_UART_RX
+Text Notes 5710 750  0    100  ~ 20
+8 Bit High Performance Microcontroller
 $EndSCHEMATC

Commit message: Switched back to TQFP micro package, placed lots of aux circuits, grid drivers, anode drivers
Parts:
- removed U301: PIC18LF67K40-I_MR, Housings_DFN_QFN:QFN-64-1EP_9x9mm_Pitch0.5mm, symbol Custom_Library:PIC18(L)F67K40-I_MR
- added U301: PIC18LF67K40-I_PT, Housings_QFP:TQFP-64_10x10mm_Pitch0.5mm, symbol Custom_Library:PIC18(L)F67K40-I_PT
Connections:
- wire segments 47 -> 46
Changed lines of the file:
@@
 Text GLabel 3760 1330 0    60   Input ~ 0
 POS24_ADC
-$Comp
-L power:GND #PWR0310
-U 1 1 5A4D9A45
-P 5010 4960
-F 0 "#PWR0310" H 5010 4710 50  0001 C CNN
-F 1 "GND" H 5010 4810 50  0000 C CNN
-F 2 "" H 5010 4960 50  0001 C CNN
-F 3 "" H 5010 4960 50  0001 C CNN
-	1    5010 4960
-	1    0    0    -1
-$EndComp
 Wire Wire Line
 	5010 900  5010 940
@@
 Text GLabel 3760 3430 0    40   Input ~ 0
 ~POS3P3_UV
-Wire Wire Line
-	5010 4960 5010 4920
-Wire Wire Line
-	5010 4920 5110 4920
-Wire Wire Line
-	5110 4920 5110 4880
-Connection ~ 5010 4920
-Wire Wire Line
-	5010 4920 5010 4880
-Wire Wire Line
-	5010 4920 4910 4920
-Wire Wire Line
-	4910 4920 4910 4880
 Text GLabel 3760 3530 0    60   Output ~ 0
 ACCUM
-$Comp
-L Custom_Library:PIC18(L)F67K40-I_MR U301
-U 1 1 5B5806FA
-P 5010 2980
-F 0 "U301" H 6060 1180 50  0000 R CNN
-F 1 "PIC18LF67K40-I_MR" H 5010 3030 50  0000 C CNN
-F 2 "Housings_DFN_QFN:QFN-64-1EP_9x9mm_Pitch0.5mm" H 5010 5080 50  0001 C CNN
-F 3 "" H 4360 3630 50  0001 C CNN
-F 4 "PIC18LF67K40T-I/MRCT-ND" H 5010 2980 50  0001 C CNN "Digi-Key PN"
-	1    5010 2980
-	1    0    0    -1
-$EndComp
 Text GLabel 3760 3630 0    60   Output ~ 0
 REF_CLK
@@
 Text Notes 5710 750  0    100  ~ 20
 8 Bit High Performance Microcontroller
+$Comp
+L Custom_Library:PIC18(L)F67K40-I_PT U301
+U 1 1 5B668926
+P 5010 2980
+F 0 "U301" H 6060 1180 50  0000 R CNN
+F 1 "PIC18LF67K40-I_PT" H 5010 3030 50  0000 C CNN
+F 2 "Housings_QFP:TQFP-64_10x10mm_Pitch0.5mm" H 5010 5080 50  0001 C CNN
+F 3 "" H 4360 3630 50  0001 C CNN
+F 4 "PIC18LF67K40T-I/PTCT-ND" H 5010 2980 50  0001 C CNN "Digi-Key PN"
+	1    5010 2980
+	1    0    0    -1
+$EndComp
+$Comp
+L power:GND #PWR?
+U 1 1 5B66A6B7
+P 5010 4960
+F 0 "#PWR?" H 5010 4710 50  0001 C CNN
+F 1 "GND" H 5010 4810 50  0000 C CNN
+F 2 "" H 5010 4960 50  0001 C CNN
+F 3 "" H 5010 4960 50  0001 C CNN
+	1    5010 4960
+	1    0    0    -1
+$EndComp
+Wire Wire Line
+	5010 4960 5010 4920
+Wire Wire Line
+	5010 4920 4960 4920
+Wire Wire Line
+	4960 4920 4960 4880
+Wire Wire Line
+	5010 4920 5060 4920
+Wire Wire Line
+	5060 4920 5060 4880
+Connection ~ 5010 4920
 $EndSCHEMATC

Commit message: Added diff pair signal names, assigned design rules to obvious nets
Connections:
- net labels added: uC_SOSC+, uC_SOSC-
- net labels removed: uC_SOSC1, uC_SOSC2
Changed lines of the file:
@@
 VFF_RUN
 Text GLabel 8130 5520 1    60   UnSpc ~ 0
-uC_SOSC2
+uC_SOSC-
 Text GLabel 7430 5520 1    60   UnSpc ~ 0
-uC_SOSC1
+uC_SOSC+
 $Comp
 L Custom-Library:C_Custom C308
@@
 Connection ~ 8130 5600
 Text GLabel 3760 3130 0    60   UnSpc ~ 0
-uC_SOSC1
+uC_SOSC+
 Text GLabel 3760 3030 0    60   UnSpc ~ 0
-uC_SOSC2
+uC_SOSC-
 $Comp
 L Custom-Library:+3.3V_MNG #PWR0309
