File: AnodeDrivers.sch (KiCad schematic (older format))
At the start: 48 parts, among them Q1101 BC847W, Q1102 BC847W, Q1103 BC856W, Q1104 BC856W, Q1105 BC847W, Q1106 BC847W, Q1107 BC856W, Q1108 BC856W, Q1109 BC847W, Q1110 BC847W, Q1111 BC856W, Q1112 BC856W, Q1113 BC847W, Q1114 BC847W, Q1115 BC856W, Q1116 BC856W

Commit message: Resolved an issue with the field names of resistors on anode and grid driver sheets
Parts:
- R1101, R1102, R1103, R1104, R1105, R1106, R1107, R1108, R1109, R1110, R1111, R1112, R1113, R1114, R1115, R1116, R1117, R1118, R1119, R1120, R1121, R1122, R1123, R1124, R1125, R1126, R1127, R1128, R1129, R1130, R1131, R1132: footprint Resistors_SMD:R_1218 -> Resistors_SMD:R_0603; display_footprint (none) -> 0603; footprint_display 0603 -> (none)
Connections:
- wire segments 48 -> 64

Commit message: Added a bunch of Digi-Key PN's
Parts:
- Q1103, Q1104, Q1107, Q1108, Q1111, Q1112, Q1115, Q1116: Digi-Key PN (none) -> 1727-4865-1-ND
- R1101, R1102, R1109, R1110, R1117, R1118, R1125, R1126: Digi-Key PN (none) -> 541-10.0KHCT-ND
- R1103, R1105, R1111, R1113, R1119, R1121, R1127, R1129: Digi-Key PN (none) -> P220KHCT-ND
- R1104, R1106, R1112, R1114, R1120, R1122, R1128, R1130: Digi-Key PN (none) -> P68KDBCT-ND
- R1107, R1108, R1115, R1116, R1123, R1124, R1131, R1132: Digi-Key PN (none) -> P16019CT-ND
Changed lines of the file:
@@
 F 2 "TO_SOT_Packages_SMD:SOT-323" H 2580 1845 50  0001 L CIN
 F 3 "" H 2380 1920 50  0001 L CNN
+F 4 "1727-4865-1-ND" H 0   0   50  0001 C CNN "Digi-Key PN"
 	1    2380 1920
 	1    0    0    1
@@
 F 5 "1/10W" H 2000 1590 50  0000 R CNN "Wattage"
 F 6 "0603" H 2000 1780 50  0000 R CNN "display_footprint"
+F 7 "P220KHCT-ND" H 0   0   50  0001 C CNN "Digi-Key PN"
 	1    2100 1690
 	1    0    0    -1
@@
 F 5 "1/10W" H 2000 2050 50  0000 R CNN "Wattage"
 F 6 "0603" H 2010 2230 50  0000 R CNN "display_footprint"
+F 7 "P68KDBCT-ND" H 0   0   50  0001 C CNN "Digi-Key PN"
 	1    2100 2150
 	1    0    0    -1
@@
 F 5 "1/10W" V 1340 2500 50  0000 C CNN "Wattage"
 F 6 "0603" V 1260 2500 50  0000 C CNN "display_footprint"
+F 7 "541-10.0KHCT-ND" H 0   0   50  0001 C CNN "Digi-Key PN"
 	1    1440 2500
 	0    -1   -1   0
@@
 F 2 "TO_SOT_Packages_SMD:SOT-323" H 4910 1845 50  0001 L CIN
 F 3 "" H 4710 1920 50  0001 L CNN
+F 4 "1727-4865-1-ND" H 0   0   50  0001 C CNN "Digi-Key PN"
 	1    4710 1920
 	1    0    0    1
@@
 F 2 "TO_SOT_Packages_SMD:SOT-323" H 9650 1845 50  0001 L CIN
 F 3 "" H 9450 1920 50  0001 L CNN
+F 4 "1727-4865-1-ND" H 0   0   50  0001 C CNN "Digi-Key PN"
 	1    9450 1920
 	1    0    0    1
@@
 F 2 "TO_SOT_Packages_SMD:SOT-323" H 2580 4175 50  0001 L CIN
 F 3 "" H 2380 4250 50  0001 L CNN
+F 4 "1727-4865-1-ND" H 0   0   50  0001 C CNN "Digi-Key PN"
 	1    2380 4250
 	1    0    0    1
@@
 F 2 "TO_SOT_Packages_SMD:SOT-323" H 4910 4175 50  0001 L CIN
 F 3 "" H 4710 4250 50  0001 L CNN
+F 4 "1727-4865-1-ND" H 0   0   50  0001 C CNN "Digi-Key PN"
 	1    4710 4250
 	1    0    0    1
@@
 F 2 "TO_SOT_Packages_SMD:SOT-323" H 7320 4175 50  0001 L CIN
 F 3 "" H 7120 4250 50  0001 L CNN
+F 4 "1727-4865-1-ND" H 0   0   50  0001 C CNN "Digi-Key PN"
 	1    7120 4250
 	1    0    0    1
@@
 F 2 "TO_SOT_Packages_SMD:SOT-323" H 9650 4175 50  0001 L CIN
 F 3 "" H 9450 4250 50  0001 L CNN
+F 4 "1727-4865-1-ND" H 0   0   50  0001 C CNN "Digi-Key PN"
 	1    9450 4250
 	1    0    0    1
@@
 F 5 "1/10W" H 2380 2450 50  0000 R CNN "Wattage"
 F 6 "0603" H 2380 2630 50  0000 R CNN "display_footprint"
+F 7 "P16019CT-ND" H 0   0   50  0001 C CNN "Digi-Key PN"
 	1    2480 2550
 	-1   0    0    -1
@@
 F 5 "1/10W" V 3670 2500 50  0000 C CNN "Wattage"
 F 6 "0603" V 3590 2500 50  0000 C CNN "display_footprint"
+F 7 "541-10.0KHCT-ND" H 0   0   50  0001 C CNN "Digi-Key PN"
 	1    3770 2500
 	0    -1   -1   0
@@
 F 5 "1/10W" V 6080 2500 50  0000 C CNN "Wattage"
 F 6 "0603" V 6000 2500 50  0000 C CNN "display_footprint"
+F 7 "541-10.0KHCT-ND" H 0   0   50  0001 C CNN "Digi-Key PN"
 	1    6180 2500
 	0    -1   -1   0
@@
 F 5 "1/10W" V 8410 2500 50  0000 C CNN "Wattage"
 F 6 "0603" V 8330 2500 50  0000 C CNN "display_footprint"
+F 7 "541-10.0KHCT-ND" H 0   0   50  0001 C CNN "Digi-Key PN"
 	1    8510 2500
 	0    -1   -1   0
@@
 F 5 "1/10W" V 8410 4830 50  0000 C CNN "Wattage"
 F 6 "0603" V 8330 4830 50  0000 C CNN "display_footprint"
+F 7 "541-10.0KHCT-ND" H 0   0   50  0001 C CNN "Digi-Key PN"
 	1    8510 4830
 	0    -1   -1   0
@@
 F 5 "1/10W" V 6080 4830 50  0000 C CNN "Wattage"
 F 6 "0603" V 6000 4830 50  0000 C CNN "display_footprint"
+F 7 "541-10.0KHCT-ND" H 0   0   50  0001 C CNN "Digi-Key PN"
 	1    6180 4830
 	0    -1   -1   0
@@
 F 5 "1/10W" V 3670 4830 50  0000 C CNN "Wattage"
 F 6 "0603" V 3590 4830 50  0000 C CNN "display_footprint"
+F 7 "541-10.0KHCT-ND" H 0   0   50  0001 C CNN "Digi-Key PN"
 	1    3770 4830
 	0    -1   -1   0
@@
 F 5 "1/10W" V 1340 4830 50  0000 C CNN "Wattage"
 F 6 "0603" V 1260 4830 50  0000 C CNN "display_footprint"
+F 7 "541-10.0KHCT-ND" H 0   0   50  0001 C CNN "Digi-Key PN"
 	1    1440 4830
 	0    -1   -1   0
@@
 F 5 "1/10W" H 4330 1590 50  0000 R CNN "Wattage"
 F 6 "0603" H 4340 1780 50  0000 R CNN "display_footprint"
+F 7 "P220KHCT-ND" H 0   0   50  0001 C CNN "Digi-Key PN"
 	1    4430 1690
 	1    0    0    -1
@@
 F 5 "1/10W" H 6740 1590 50  0000 R CNN "Wattage"
 F 6 "0603" H 6750 1780 50  0000 R CNN "display_footprint"
+F 7 "P220KHCT-ND" H 0   0   50  0001 C CNN "Digi-Key PN"
 	1    6840 1690
 	1    0    0    -1
@@
 F 5 "1/10W" H 9070 1590 50  0000 R CNN "Wattage"
 F 6 "0603" H 9080 1780 50  0000 R CNN "display_footprint"
+F 7 "P220KHCT-ND" H 0   0   50  0001 C CNN "Digi-Key PN"
 	1    9170 1690
 	1    0    0    -1
@@
 F 5 "1/10W" H 9070 3920 50  0000 R CNN "Wattage"
 F 6 "0603" H 9080 4110 50  0000 R CNN "display_footprint"
+F 7 "P220KHCT-ND" H 0   0   50  0001 C CNN "Digi-Key PN"
 	1    9170 4020
 	1    0    0    -1
@@
 F 5 "1/10W" H 6740 3920 50  0000 R CNN "Wattage"
 F 6 "0603" H 6750 4110 50  0000 R CNN "display_footprint"
+F 7 "P220KHCT-ND" H 0   0   50  0001 C CNN "Digi-Key PN"
 	1    6840 4020
 	1    0    0    -1
@@
 F 5 "1/10W" H 4330 3920 50  0000 R CNN "Wattage"
 F 6 "0603" H 4330 4110 50  0000 R CNN "display_footprint"
+F 7 "P220KHCT-ND" H 0   0   50  0001 C CNN "Digi-Key PN"
 	1    4430 4020
 	1    0    0    -1
@@
 F 5 "1/10W" H 2000 3920 50  0000 R CNN "Wattage"
 F 6 "0603" H 2010 4100 50  0000 R CNN "display_footprint"
+F 7 "P220KHCT-ND" H 0   0   50  0001 C CNN "Digi-Key PN"
 	1    2100 4020
 	1    0    0    -1
@@
 F 2 "TO_SOT_Packages_SMD:SOT-323" H 7320 1845 50  0001 L CIN
 F 3 "" H 7120 1920 50  0001 L CNN
+F 4 "1727-4865-1-ND" H 0   0   50  0001 C CNN "Digi-Key PN"
 	1    7120 1920
 	1    0    0    1
@@
 F 5 "1/10W" H 4330 2050 50  0000 R CNN "Wattage"
 F 6 "0603" H 4340 2230 50  0000 R CNN "display_footprint"
+F 7 "P68KDBCT-ND" H 0   0   50  0001 C CNN "Digi-Key PN"
 	1    4430 2150
 	1    0    0    -1
@@
 F 5 "1/10W" H 6740 2050 50  0000 R CNN "Wattage"
 F 6 "0603" H 6750 2240 50  0000 R CNN "display_footprint"
+F 7 "P68KDBCT-ND" H 0   0   50  0001 C CNN "Digi-Key PN"
 	1    6840 2150
 	1    0    0    -1
@@
 F 5 "0603" H 9070 2240 50  0000 R CNN "display_footprint"
 F 6 "1%" H 9080 2150 50  0000 R CNN "Tolerance"
+F 7 "P68KDBCT-ND" H 0   0   50  0001 C CNN "Digi-Key PN"
 	1    9170 2150
 	1    0    0    -1
@@
 F 5 "1/10W" H 9070 4380 50  0000 R CNN "Wattage"
 F 6 "0603" H 9080 4570 50  0000 R CNN "display_footprint"
+F 7 "P68KDBCT-ND" H 0   0   50  0001 C CNN "Digi-Key PN"
 	1    9170 4480
 	1    0    0    -1
@@
 F 5 "1/10W" H 6740 4380 50  0000 R CNN "Wattage"
 F 6 "0603" H 6750 4560 50  0000 R CNN "display_footprint"
+F 7 "P68KDBCT-ND" H 0   0   50  0001 C CNN "Digi-Key PN"
 	1    6840 4480
 	1    0    0    -1
@@
 F 5 "1/10W" H 4330 4380 50  0000 R CNN "Wattage"
 F 6 "0603" H 4340 4570 50  0000 R CNN "display_footprint"
+F 7 "P68KDBCT-ND" H 0   0   50  0001 C CNN "Digi-Key PN"
 	1    4430 4480
 	1    0    0    -1
@@
 F 5 "1/10W" H 2000 4380 50  0000 R CNN "Wattage"
 F 6 "0603" H 2010 4570 50  0000 R CNN "display_footprint"
+F 7 "P68KDBCT-ND" H 0   0   50  0001 C CNN "Digi-Key PN"
 	1    2100 4480
 	1    0    0    -1
@@
 F 5 "1/10W" H 4710 2450 50  0000 R CNN "Wattage"
 F 6 "0603" H 4710 2640 50  0000 R CNN "display_footprint"
+F 7 "P16019CT-ND" H 0   0   50  0001 C CNN "Digi-Key PN"
 	1    4810 2550
 	-1   0    0    -1
@@
 F 5 "1/10W" H 7120 2450 50  0000 R CNN "Wattage"
 F 6 "0603" H 7120 2640 50  0000 R CNN "display_footprint"
+F 7 "P16019CT-ND" H 0   0   50  0001 C CNN "Digi-Key PN"
 	1    7220 2550
 	-1   0    0    -1
@@
 F 5 "1/10W" H 9450 2450 50  0000 R CNN "Wattage"
 F 6 "0603" H 9450 2640 50  0000 R CNN "display_footprint"
+F 7 "P16019CT-ND" H 0   0   50  0001 C CNN "Digi-Key PN"
 	1    9550 2550
 	-1   0    0    -1
@@
 F 5 "1/10W" H 9450 4780 50  0000 R CNN "Wattage"
 F 6 "0603" H 9450 4970 50  0000 R CNN "display_footprint"
+F 7 "P16019CT-ND" H 0   0   50  0001 C CNN "Digi-Key PN"
 	1    9550 4880
 	-1   0    0    -1
@@
 F 5 "1/10W" H 7120 4780 50  0000 R CNN "Wattage"
 F 6 "0603" H 7120 4970 50  0000 R CNN "display_footprint"
+F 7 "P16019CT-ND" H 0   0   50  0001 C CNN "Digi-Key PN"
 	1    7220 4880
 	-1   0    0    -1
@@
 F 5 "1/10W" H 4710 4780 50  0000 R CNN "Wattage"
 F 6 "0603" H 4710 4960 50  0000 R CNN "display_footprint"
+F 7 "P16019CT-ND" H 0   0   50  0001 C CNN "Digi-Key PN"
 	1    4810 4880
 	-1   0    0    -1
@@
 F 5 "1/10W" H 2380 4780 50  0000 R CNN "Wattage"
 F 6 "0603" H 2380 4960 50  0000 R CNN "display_footprint"
+F 7 "P16019CT-ND" H 0   0   50  0001 C CNN "Digi-Key PN"
 	1    2480 4880
 	-1   0    0    -1

Commit message: Arranged more components on PCB, cleaned up schematic, added page titles, finished finding DigiKey PN's
Parts:
- Q1101, Q1102, Q1105, Q1106, Q1109, Q1110, Q1113, Q1114: value BC847W -> PMSTA06; Digi-Key PN (none) -> 1727-6293-1-ND
- R1101, R1102, R1109, R1110, R1117, R1118, R1125, R1126: Digi-Key PN 541-10.0KHCT-ND -> P10.0KHCT-ND
Other:
- note added: "Anode Drivers"
Changed lines of the file:
@@
 U 1 1 5A2D344E
 P 2000 2500
-F 0 "Q1101" H 2200 2575 50  0000 L CNN
-F 1 "BC847W" H 1640 2610 50  0000 L CNN
+F 0 "Q1101" H 2180 2620 50  0000 L CNN
+F 1 "PMSTA06" H 1640 2610 50  0000 L CNN
 F 2 "TO_SOT_Packages_SMD:SOT-323" H 2200 2425 50  0001 L CIN
 F 3 "" H 2000 2500 50  0001 L CNN
+F 4 "1727-6293-1-ND" H 0   0   50  0001 C CNN "Digi-Key PN"
 	1    2000 2500
 	1    0    0    -1
@@
 F 5 "1/10W" V 1340 2500 50  0000 C CNN "Wattage"
 F 6 "0603" V 1260 2500 50  0000 C CNN "display_footprint"
-F 7 "541-10.0KHCT-ND" H 0   0   50  0001 C CNN "Digi-Key PN"
+F 7 "P10.0KHCT-ND" H 0   0   50  0001 C CNN "Digi-Key PN"
 	1    1440 2500
 	0    -1   -1   0
@@
 U 1 1 5A2D6BEB
 P 4330 2500
-F 0 "Q1105" H 4530 2575 50  0000 L CNN
-F 1 "BC847W" H 3970 2610 50  0000 L CNN
+F 0 "Q1105" H 4500 2610 50  0000 L CNN
+F 1 "PMSTA06" H 3970 2610 50  0000 L CNN
 F 2 "TO_SOT_Packages_SMD:SOT-323" H 4530 2425 50  0001 L CIN
 F 3 "" H 4330 2500 50  0001 L CNN
+F 4 "1727-6293-1-ND" H 0   0   50  0001 C CNN "Digi-Key PN"
 	1    4330 2500
 	1    0    0    -1
@@
 U 1 1 5A2D6DCF
 P 6740 2500
-F 0 "Q1109" H 6940 2575 50  0000 L CNN
-F 1 "BC847W" H 6380 2610 50  0000 L CNN
+F 0 "Q1109" H 6920 2600 50  0000 L CNN
+F 1 "PMSTA06" H 6380 2610 50  0000 L CNN
 F 2 "TO_SOT_Packages_SMD:SOT-323" H 6940 2425 50  0001 L CIN
 F 3 "" H 6740 2500 50  0001 L CNN
+F 4 "1727-6293-1-ND" H 0   0   50  0001 C CNN "Digi-Key PN"
 	1    6740 2500
 	1    0    0    -1
@@
 U 1 1 5A2D6F29
 P 9070 2500
-F 0 "Q1113" H 9270 2575 50  0000 L CNN
-F 1 "BC847W" H 8710 2610 50  0000 L CNN
+F 0 "Q1113" H 9250 2620 50  0000 L CNN
+F 1 "PMSTA06" H 8710 2610 50  0000 L CNN
 F 2 "TO_SOT_Packages_SMD:SOT-323" H 9270 2425 50  0001 L CIN
 F 3 "" H 9070 2500 50  0001 L CNN
+F 4 "1727-6293-1-ND" H 0   0   50  0001 C CNN "Digi-Key PN"
 	1    9070 2500
 	1    0    0    -1
@@
 U 1 1 5A2D851C
 P 2000 4830
-F 0 "Q1102" H 2200 4905 50  0000 L CNN
-F 1 "BC847W" H 1640 4940 50  0000 L CNN
+F 0 "Q1102" H 2180 4960 50  0000 L CNN
+F 1 "PMSTA06" H 1640 4940 50  0000 L CNN
 F 2 "TO_SOT_Packages_SMD:SOT-323" H 2200 4755 50  0001 L CIN
 F 3 "" H 2000 4830 50  0001 L CNN
+F 4 "1727-6293-1-ND" H 0   0   50  0001 C CNN "Digi-Key PN"
 	1    2000 4830
 	1    0    0    -1
@@
 U 1 1 5A2D856E
 P 4330 4830
-F 0 "Q1106" H 4530 4905 50  0000 L CNN
-F 1 "BC847W" H 3970 4940 50  0000 L CNN
+F 0 "Q1106" H 4510 4950 50  0000 L CNN
+F 1 "PMSTA06" H 3970 4940 50  0000 L CNN
 F 2 "TO_SOT_Packages_SMD:SOT-323" H 4530 4755 50  0001 L CIN
 F 3 "" H 4330 4830 50  0001 L CNN
+F 4 "1727-6293-1-ND" H 0   0   50  0001 C CNN "Digi-Key PN"
 	1    4330 4830
 	1    0    0    -1
@@
 U 1 1 5A2D85C0
 P 6740 4830
-F 0 "Q1110" H 6940 4905 50  0000 L CNN
-F 1 "BC847W" H 6380 4940 50  0000 L CNN
+F 0 "Q1110" H 6920 4960 50  0000 L CNN
+F 1 "PMSTA06" H 6380 4940 50  0000 L CNN
 F 2 "TO_SOT_Packages_SMD:SOT-323" H 6940 4755 50  0001 L CIN
 F 3 "" H 6740 4830 50  0001 L CNN
+F 4 "1727-6293-1-ND" H 0   0   50  0001 C CNN "Digi-Key PN"
 	1    6740 4830
 	1    0    0    -1
@@
 U 1 1 5A2D8612
 P 9070 4830
-F 0 "Q1114" H 9270 4905 50  0000 L CNN
-F 1 "BC847W" H 8710 4940 50  0000 L CNN
+F 0 "Q1114" H 9250 4950 50  0000 L CNN
+F 1 "PMSTA06" H 8710 4940 50  0000 L CNN
 F 2 "TO_SOT_Packages_SMD:SOT-323" H 9270 4755 50  0001 L CIN
 F 3 "" H 9070 4830 50  0001 L CNN
+F 4 "1727-6293-1-ND" H 0   0   50  0001 C CNN "Digi-Key PN"
 	1    9070 4830
 	1    0    0    -1
@@
 F 5 "1/10W" V 3670 2500 50  0000 C CNN "Wattage"
 F 6 "0603" V 3590 2500 50  0000 C CNN "display_footprint"
-F 7 "541-10.0KHCT-ND" H 0   0   50  0001 C CNN "Digi-Key PN"
+F 7 "P10.0KHCT-ND" H 0   0   50  0001 C CNN "Digi-Key PN"
 	1    3770 2500
 	0    -1   -1   0
@@
 F 5 "1/10W" V 6080 2500 50  0000 C CNN "Wattage"
 F 6 "0603" V 6000 2500 50  0000 C CNN "display_footprint"
-F 7 "541-10.0KHCT-ND" H 0   0   50  0001 C CNN "Digi-Key PN"
+F 7 "P10.0KHCT-ND" H 0   0   50  0001 C CNN "Digi-Key PN"
 	1    6180 2500
 	0    -1   -1   0
@@
 F 5 "1/10W" V 8410 2500 50  0000 C CNN "Wattage"
 F 6 "0603" V 8330 2500 50  0000 C CNN "display_footprint"
-F 7 "541-10.0KHCT-ND" H 0   0   50  0001 C CNN "Digi-Key PN"
+F 7 "P10.0KHCT-ND" H 0   0   50  0001 C CNN "Digi-Key PN"
 	1    8510 2500
 	0    -1   -1   0
@@
 F 5 "1/10W" V 8410 4830 50  0000 C CNN "Wattage"
 F 6 "0603" V 8330 4830 50  0000 C CNN "display_footprint"
-F 7 "541-10.0KHCT-ND" H 0   0   50  0001 C CNN "Digi-Key PN"
+F 7 "P10.0KHCT-ND" H 0   0   50  0001 C CNN "Digi-Key PN"
 	1    8510 4830
 	0    -1   -1   0
@@
 F 5 "1/10W" V 6080 4830 50  0000 C CNN "Wattage"
 F 6 "0603" V 6000 4830 50  0000 C CNN "display_footprint"
-F 7 "541-10.0KHCT-ND" H 0   0   50  0001 C CNN "Digi-Key PN"
+F 7 "P10.0KHCT-ND" H 0   0   50  0001 C CNN "Digi-Key PN"
 	1    6180 4830
 	0    -1   -1   0
@@
 F 5 "1/10W" V 3670 4830 50  0000 C CNN "Wattage"
 F 6 "0603" V 3590 4830 50  0000 C CNN "display_footprint"
-F 7 "541-10.0KHCT-ND" H 0   0   50  0001 C CNN "Digi-Key PN"
+F 7 "P10.0KHCT-ND" H 0   0   50  0001 C CNN "Digi-Key PN"
 	1    3770 4830
 	0    -1   -1   0
@@
 F 5 "1/10W" V 1340 4830 50  0000 C CNN "Wattage"
 F 6 "0603" V 1260 4830 50  0000 C CNN "display_footprint"
-F 7 "541-10.0KHCT-ND" H 0   0   50  0001 C CNN "Digi-Key PN"
+F 7 "P10.0KHCT-ND" H 0   0   50  0001 C CNN "Digi-Key PN"
 	1    1440 4830
 	0    -1   -1   0
@@
 Wire Wire Line
 	9550 4590 9550 4450
+Text Notes 5220 910  0    100  ~ 20
+Anode Drivers
 $EndSCHEMATC
