File: GridDrivers.sch (KiCad schematic (older format))
At the start: 36 parts, among them Q1201 BC847W, Q1202 BC847W, Q1203 BC856W, Q1204 BC856W, Q1205 BC847W, Q1206 BC847W, Q1207 BC856W, Q1208 BC856W, Q1209 BC847W, Q1210 BC847W, Q1211 BC856W, Q1212 BC856W

Commit message: Resolved an issue with the field names of resistors on anode and grid driver sheets
Parts:
- R1201, R1202, R1203, R1204, R1205, R1206, R1207, R1208, R1209, R1210, R1211, R1212, R1213, R1214, R1215, R1216, R1217, R1218, R1219, R1220, R1221, R1222, R1223, R1224: footprint Resistors_SMD:R_1218 -> Resistors_SMD:R_0603; display_footprint (none) -> 0603; footprint_display 0603 -> (none)
Connections:
- wire segments 36 -> 48

Commit message: Added a bunch of Digi-Key PN's
Parts:
- Q1203, Q1204, Q1207, Q1208, Q1211, Q1212: Digi-Key PN (none) -> 1727-4865-1-ND
- R1201, R1202, R1209, R1210, R1217, R1218: Digi-Key PN (none) -> 541-10.0KHCT-ND
- R1203, R1205, R1211, R1213, R1219, R1221: Digi-Key PN (none) -> P220KHCT-ND
- R1204, R1206, R1212, R1214, R1220, R1222: Digi-Key PN (none) -> P68KDBCT-ND
- R1207, R1208, R1215, R1216, R1223, R1224: Digi-Key PN (none) -> P16019CT-ND
Changed lines of the file:
@@
 F 2 "TO_SOT_Packages_SMD:SOT-323" H 2580 1845 50  0001 L CIN
 F 3 "" H 2380 1920 50  0001 L CNN
+F 4 "1727-4865-1-ND" H 0   0   50  0001 C CNN "Digi-Key PN"
 	1    2380 1920
 	1    0    0    1
@@
 F 2 "TO_SOT_Packages_SMD:SOT-323" H 4910 1845 50  0001 L CIN
 F 3 "" H 4710 1920 50  0001 L CNN
+F 4 "1727-4865-1-ND" H 0   0   50  0001 C CNN "Digi-Key PN"
 	1    4710 1920
 	1    0    0    1
@@
 F 2 "TO_SOT_Packages_SMD:SOT-323" H 7320 1845 50  0001 L CIN
 F 3 "" H 7120 1920 50  0001 L CNN
+F 4 "1727-4865-1-ND" H 0   0   50  0001 C CNN "Digi-Key PN"
 	1    7120 1920
 	1    0    0    1
@@
 F 2 "TO_SOT_Packages_SMD:SOT-323" H 2580 4175 50  0001 L CIN
 F 3 "" H 2380 4250 50  0001 L CNN
+F 4 "1727-4865-1-ND" H 0   0   50  0001 C CNN "Digi-Key PN"
 	1    2380 4250
 	1    0    0    1
@@
 F 2 "TO_SOT_Packages_SMD:SOT-323" H 4910 4175 50  0001 L CIN
 F 3 "" H 4710 4250 50  0001 L CNN
+F 4 "1727-4865-1-ND" H 0   0   50  0001 C CNN "Digi-Key PN"
 	1    4710 4250
 	1    0    0    1
@@
 F 2 "TO_SOT_Packages_SMD:SOT-323" H 7320 4175 50  0001 L CIN
 F 3 "" H 7120 4250 50  0001 L CNN
+F 4 "1727-4865-1-ND" H 0   0   50  0001 C CNN "Digi-Key PN"
 	1    7120 4250
 	1    0    0    1
@@
 F 5 "1/10W" V 1340 2500 50  0000 C CNN "Wattage"
 F 6 "0603" V 1260 2500 50  0000 C CNN "display_footprint"
+F 7 "541-10.0KHCT-ND" H 0   0   50  0001 C CNN "Digi-Key PN"
 	1    1440 2500
 	0    -1   -1   0
@@
 F 5 "1/10W" V 3670 2500 50  0000 C CNN "Wattage"
 F 6 "0603" V 3590 2500 50  0000 C CNN "display_footprint"
+F 7 "541-10.0KHCT-ND" H 0   0   50  0001 C CNN "Digi-Key PN"
 	1    3770 2500
 	0    -1   -1   0
@@
 F 5 "1/10W" V 6080 2500 50  0000 C CNN "Wattage"
 F 6 "0603" V 6000 2500 50  0000 C CNN "display_footprint"
+F 7 "541-10.0KHCT-ND" H 0   0   50  0001 C CNN "Digi-Key PN"
 	1    6180 2500
 	0    -1   -1   0
@@
 F 5 "1/10W" V 6080 4830 50  0000 C CNN "Wattage"
 F 6 "0603" V 6000 4830 50  0000 C CNN "display_footprint"
+F 7 "541-10.0KHCT-ND" H 0   0   50  0001 C CNN "Digi-Key PN"
 	1    6180 4830
 	0    -1   -1   0
@@
 F 5 "1/10W" V 3670 4830 50  0000 C CNN "Wattage"
 F 6 "0603" V 3590 4830 50  0000 C CNN "display_footprint"
+F 7 "541-10.0KHCT-ND" H 0   0   50  0001 C CNN "Digi-Key PN"
 	1    3770 4830
 	0    -1   -1   0
@@
 F 5 "1/10W" V 1340 4830 50  0000 C CNN "Wattage"
 F 6 "0603" V 1260 4830 50  0000 C CNN "display_footprint"
+F 7 "541-10.0KHCT-ND" H 0   0   50  0001 C CNN "Digi-Key PN"
 	1    1440 4830
 	0    -1   -1   0
@@
 F 5 "1/10W" H 2000 1590 50  0000 R CNN "Wattage"
 F 6 "0603" H 2010 1780 50  0000 R CNN "display_footprint"
+F 7 "P220KHCT-ND" H 0   0   50  0001 C CNN "Digi-Key PN"
 	1    2100 1690
 	1    0    0    -1
@@
 F 5 "1/10W" H 4330 1590 50  0000 R CNN "Wattage"
 F 6 "0603" H 4340 1770 50  0000 R CNN "display_footprint"
+F 7 "P220KHCT-ND" H 0   0   50  0001 C CNN "Digi-Key PN"
 	1    4430 1690
 	1    0    0    -1
@@
 F 5 "1/10W" H 6740 1590 50  0000 R CNN "Wattage"
 F 6 "0603" H 6750 1780 50  0000 R CNN "display_footprint"
+F 7 "P220KHCT-ND" H 0   0   50  0001 C CNN "Digi-Key PN"
 	1    6840 1690
 	1    0    0    -1
@@
 F 5 "1/10W" H 6740 3920 50  0000 R CNN "Wattage"
 F 6 "0603" H 6750 4110 50  0000 R CNN "display_footprint"
+F 7 "P220KHCT-ND" H 0   0   50  0001 C CNN "Digi-Key PN"
 	1    6840 4020
 	1    0    0    -1
@@
 F 5 "1/10W" H 4330 3920 50  0000 R CNN "Wattage"
 F 6 "0603" H 4330 4110 50  0000 R CNN "display_footprint"
+F 7 "P220KHCT-ND" H 0   0   50  0001 C CNN "Digi-Key PN"
 	1    4430 4020
 	1    0    0    -1
@@
 F 5 "1/10W" H 2000 3920 50  0000 R CNN "Wattage"
 F 6 "0603" H 2010 4110 50  0000 R CNN "display_footprint"
+F 7 "P220KHCT-ND" H 0   0   50  0001 C CNN "Digi-Key PN"
 	1    2100 4020
 	1    0    0    -1
@@
 F 5 "1/10W" H 2000 2050 50  0000 R CNN "Wattage"
 F 6 "0603" H 2010 2240 50  0000 R CNN "display_footprint"
+F 7 "P68KDBCT-ND" H 0   0   50  0001 C CNN "Digi-Key PN"
 	1    2100 2150
 	1    0    0    -1
@@
 F 5 "1/10W" H 4330 2050 50  0000 R CNN "Wattage"
 F 6 "0603" H 4330 2230 50  0000 R CNN "display_footprint"
+F 7 "P68KDBCT-ND" H 0   0   50  0001 C CNN "Digi-Key PN"
 	1    4430 2150
 	1    0    0    -1
@@
 F 5 "1/10W" H 6740 2050 50  0000 R CNN "Wattage"
 F 6 "0603" H 6750 2240 50  0000 R CNN "display_footprint"
+F 7 "P68KDBCT-ND" H 0   0   50  0001 C CNN "Digi-Key PN"
 	1    6840 2150
 	1    0    0    -1
@@
 F 5 "1/10W" H 6740 4380 50  0000 R CNN "Wattage"
 F 6 "0603" H 6750 4570 50  0000 R CNN "display_footprint"
+F 7 "P68KDBCT-ND" H 0   0   50  0001 C CNN "Digi-Key PN"
 	1    6840 4480
 	1    0    0    -1
@@
 F 5 "1/10W" H 4330 4380 50  0000 R CNN "Wattage"
 F 6 "0603" H 4330 4560 50  0000 R CNN "display_footprint"
+F 7 "P68KDBCT-ND" H 0   0   50  0001 C CNN "Digi-Key PN"
 	1    4430 4480
 	1    0    0    -1
@@
 F 5 "1/10W" H 2000 4380 50  0000 R CNN "Wattage"
 F 6 "0603" H 2010 4570 50  0000 R CNN "display_footprint"
+F 7 "P68KDBCT-ND" H 0   0   50  0001 C CNN "Digi-Key PN"
 	1    2100 4480
 	1    0    0    -1
@@
 F 5 "1/10W" H 2380 2450 50  0000 R CNN "Wattage"
 F 6 "0603" H 2380 2640 50  0000 R CNN "display_footprint"
+F 7 "P16019CT-ND" H 0   0   50  0001 C CNN "Digi-Key PN"
 	1    2480 2550
 	-1   0    0    -1
@@
 F 5 "1/10W" H 4710 2450 50  0000 R CNN "Wattage"
 F 6 "0603" H 4710 2640 50  0000 R CNN "display_footprint"
+F 7 "P16019CT-ND" H 0   0   50  0001 C CNN "Digi-Key PN"
 	1    4810 2550
 	-1   0    0    -1
@@
 F 5 "1/10W" H 7120 2450 50  0000 R CNN "Wattage"
 F 6 "0603" H 7120 2640 50  0000 R CNN "display_footprint"
+F 7 "P16019CT-ND" H 0   0   50  0001 C CNN "Digi-Key PN"
 	1    7220 2550
 	-1   0    0    -1
@@
 F 5 "1/10W" H 7120 4780 50  0000 R CNN "Wattage"
 F 6 "0603" H 7120 4970 50  0000 R CNN "display_footprint"
+F 7 "P16019CT-ND" H 0   0   50  0001 C CNN "Digi-Key PN"
 	1    7220 4880
 	-1   0    0    -1
@@
 F 5 "1/10W" H 4710 4780 50  0000 R CNN "Wattage"
 F 6 "0603" H 4710 4980 50  0000 R CNN "display_footprint"
+F 7 "P16019CT-ND" H 0   0   50  0001 C CNN "Digi-Key PN"
 	1    4810 4880
 	-1   0    0    -1
@@
 F 5 "1/10W" H 2380 4780 50  0000 R CNN "Wattage"
 F 6 "0603" H 2380 4960 50  0000 R CNN "display_footprint"
+F 7 "P16019CT-ND" H 0   0   50  0001 C CNN "Digi-Key PN"
 	1    2480 4880
 	-1   0    0    -1

Commit message: Arranged more components on PCB, cleaned up schematic, added page titles, finished finding DigiKey PN's
Parts:
- Q1201, Q1202, Q1205, Q1206, Q1209, Q1210: value BC847W -> PMSTA06; Digi-Key PN (none) -> 1727-6293-1-ND
- R1201, R1202, R1209, R1210, R1217, R1218: Digi-Key PN 541-10.0KHCT-ND -> P10.0KHCT-ND
Other:
- note added: "Grid Drivers"
Changed lines of the file:
@@
 U 1 1 5A2FAE9E
 P 2000 2500
-F 0 "Q1201" H 2200 2575 50  0000 L CNN
-F 1 "BC847W" H 1640 2610 50  0000 L CNN
+F 0 "Q1201" H 2170 2620 50  0000 L CNN
+F 1 "PMSTA06" H 1640 2610 50  0000 L CNN
 F 2 "TO_SOT_Packages_SMD:SOT-323" H 2200 2425 50  0001 L CIN
 F 3 "" H 2000 2500 50  0001 L CNN
+F 4 "1727-6293-1-ND" H 0   0   50  0001 C CNN "Digi-Key PN"
 	1    2000 2500
 	1    0    0    -1
@@
 U 1 1 5A2FAEDF
 P 4330 2500
-F 0 "Q1205" H 4530 2575 50  0000 L CNN
-F 1 "BC847W" H 3970 2610 50  0000 L CNN
+F 0 "Q1205" H 4510 2620 50  0000 L CNN
+F 1 "PMSTA06" H 3970 2610 50  0000 L CNN
 F 2 "TO_SOT_Packages_SMD:SOT-323" H 4530 2425 50  0001 L CIN
 F 3 "" H 4330 2500 50  0001 L CNN
+F 4 "1727-6293-1-ND" H 0   0   50  0001 C CNN "Digi-Key PN"
 	1    4330 2500
 	1    0    0    -1
@@
 U 1 1 5A2FAF18
 P 6740 2500
-F 0 "Q1209" H 6940 2575 50  0000 L CNN
-F 1 "BC847W" H 6380 2610 50  0000 L CNN
+F 0 "Q1209" H 6920 2610 50  0000 L CNN
+F 1 "PMSTA06" H 6380 2610 50  0000 L CNN
 F 2 "TO_SOT_Packages_SMD:SOT-323" H 6940 2425 50  0001 L CIN
 F 3 "" H 6740 2500 50  0001 L CNN
+F 4 "1727-6293-1-ND" H 0   0   50  0001 C CNN "Digi-Key PN"
 	1    6740 2500
 	1    0    0    -1
@@
 U 1 1 5A2FAF8A
 P 2000 4830
-F 0 "Q1202" H 2200 4905 50  0000 L CNN
-F 1 "BC847W" H 1640 4940 50  0000 L CNN
+F 0 "Q1202" H 2180 4950 50  0000 L CNN
+F 1 "PMSTA06" H 1640 4940 50  0000 L CNN
 F 2 "TO_SOT_Packages_SMD:SOT-323" H 2200 4755 50  0001 L CIN
 F 3 "" H 2000 4830 50  0001 L CNN
+F 4 "1727-6293-1-ND" H 0   0   50  0001 C CNN "Digi-Key PN"
 	1    2000 4830
 	1    0    0    -1
@@
 U 1 1 5A2FAFC3
 P 4330 4830
-F 0 "Q1206" H 4530 4905 50  0000 L CNN
-F 1 "BC847W" H 3970 4940 50  0000 L CNN
+F 0 "Q1206" H 4510 4940 50  0000 L CNN
+F 1 "PMSTA06" H 3970 4940 50  0000 L CNN
 F 2 "TO_SOT_Packages_SMD:SOT-323" H 4530 4755 50  0001 L CIN
 F 3 "" H 4330 4830 50  0001 L CNN
+F 4 "1727-6293-1-ND" H 0   0   50  0001 C CNN "Digi-Key PN"
 	1    4330 4830
 	1    0    0    -1
@@
 U 1 1 5A2FAFFC
 P 6740 4830
-F 0 "Q1210" H 6940 4905 50  0000 L CNN
-F 1 "BC847W" H 6380 4940 50  0000 L CNN
+F 0 "Q1210" H 6920 4940 50  0000 L CNN
+F 1 "PMSTA06" H 6380 4940 50  0000 L CNN
 F 2 "TO_SOT_Packages_SMD:SOT-323" H 6940 4755 50  0001 L CIN
 F 3 "" H 6740 4830 50  0001 L CNN
+F 4 "1727-6293-1-ND" H 0   0   50  0001 C CNN "Digi-Key PN"
 	1    6740 4830
 	1    0    0    -1
@@
 F 5 "1/10W" V 1340 2500 50  0000 C CNN "Wattage"
 F 6 "0603" V 1260 2500 50  0000 C CNN "display_footprint"
-F 7 "541-10.0KHCT-ND" H 0   0   50  0001 C CNN "Digi-Key PN"
+F 7 "P10.0KHCT-ND" H 0   0   50  0001 C CNN "Digi-Key PN"
 	1    1440 2500
 	0    -1   -1   0
@@
 F 5 "1/10W" V 3670 2500 50  0000 C CNN "Wattage"
 F 6 "0603" V 3590 2500 50  0000 C CNN "display_footprint"
-F 7 "541-10.0KHCT-ND" H 0   0   50  0001 C CNN "Digi-Key PN"
+F 7 "P10.0KHCT-ND" H 0   0   50  0001 C CNN "Digi-Key PN"
 	1    3770 2500
 	0    -1   -1   0
@@
 F 5 "1/10W" V 6080 2500 50  0000 C CNN "Wattage"
 F 6 "0603" V 6000 2500 50  0000 C CNN "display_footprint"
-F 7 "541-10.0KHCT-ND" H 0   0   50  0001 C CNN "Digi-Key PN"
+F 7 "P10.0KHCT-ND" H 0   0   50  0001 C CNN "Digi-Key PN"
 	1    6180 2500
 	0    -1   -1   0
@@
 F 5 "1/10W" V 6080 4830 50  0000 C CNN "Wattage"
 F 6 "0603" V 6000 4830 50  0000 C CNN "display_footprint"
-F 7 "541-10.0KHCT-ND" H 0   0   50  0001 C CNN "Digi-Key PN"
+F 7 "P10.0KHCT-ND" H 0   0   50  0001 C CNN "Digi-Key PN"
 	1    6180 4830
 	0    -1   -1   0
@@
 F 5 "1/10W" V 3670 4830 50  0000 C CNN "Wattage"
 F 6 "0603" V 3590 4830 50  0000 C CNN "display_footprint"
-F 7 "541-10.0KHCT-ND" H 0   0   50  0001 C CNN "Digi-Key PN"
+F 7 "P10.0KHCT-ND" H 0   0   50  0001 C CNN "Digi-Key PN"
 	1    3770 4830
 	0    -1   -1   0
@@
 F 5 "1/10W" V 1340 4830 50  0000 C CNN "Wattage"
 F 6 "0603" V 1260 4830 50  0000 C CNN "display_footprint"
-F 7 "541-10.0KHCT-ND" H 0   0   50  0001 C CNN "Digi-Key PN"
+F 7 "P10.0KHCT-ND" H 0   0   50  0001 C CNN "Digi-Key PN"
 	1    1440 4830
 	0    -1   -1   0
@@
 Wire Wire Line
 	7220 4590 7220 4450
+Text Notes 4490 780  0    100  ~ 20
+Grid Drivers
 $EndSCHEMATC
