File: hdw/VFD_Clock/POS3P3_BCKP_Supply.sch (KiCad schematic (older format))
At the start: 0 parts

Commit message: More revisions
Parts:
- added C?: 2.2nF, Capacitors_SMD:C_0603, symbol Custom_Library:C_Custom
- added C?: 15F, Custom Footprints Library:SCCT30B156SRB, symbol Custom_Library:CP1_Alum_Custom
- added C?: 100uF, Capacitors_Tantalum_SMD:CP_Tantalum_Case-D_EIA-7343-31_Reflow, symbol Custom_Library:CP_Tant_Custom
- added C? (x2): 10uF, Capacitors_SMD:C_1206, symbol Custom_Library:C_Custom
- added JP?: ~BSTEN, Pin_Headers:Pin_Header_Straight_1x02_Pitch2.54mm, symbol Jumper:Jumper_2_Open
- added JP?: ~CHGEN, Pin_Headers:Pin_Header_Straight_1x02_Pitch2.54mm, symbol Jumper:Jumper_2_Open
- added L?: 2.2uH, Inductors_SMD:L_Vishay_IHLP-2020, symbol Custom_Library:L_Custom
- added MK? (x2): Shunt, symbol Custom_Library:Shunt
- added Q?: IPC100N04S51R7ATMA1, TO_SOT_Packages_SMD:TDSON-8-1, symbol Custom_Library:IPC100N04S51R7ATMA1
- added R?: 1k, Resistors_SMD:R_0603, symbol Custom_Library:R_Custom
- added R?: 931k, Resistors_SMD:R_0603, symbol Custom_Library:R_Custom
- added R?: 392k, Resistors_SMD:R_0603, symbol Custom_Library:R_Custom
- added R?: 1.07M, Resistors_SMD:R_0603, symbol Custom_Library:R_Custom
- added R?: 340k, Resistors_SMD:R_0603, symbol Custom_Library:R_Custom
- added R?: 12m, Resistors_SMD:R_0805, symbol Custom_Library:R_Custom
- added R?: 121k, Resistors_SMD:R_0603, symbol Custom_Library:R_Custom
- added R?: 75k, Resistors_SMD:R_0603, symbol Custom_Library:R_Custom
- added R? (x6): 1M, Resistors_SMD:R_0603, symbol Custom_Library:R_Custom
- added TP? (x2): TP, Measurement_Points:Test_Point_Keystone_5000-5004_Miniature, symbol Custom_Library:TP
- added U?: LTC4041UFD, Housings_DFN_QFN:QFN-24-1EP_4x5mm_Pitch0.5mm, symbol Custom_Library:LTC4041UFD
Connections:
- new net: R?.1, R?.2, U?.10 (RSTFB), U?.18 (BSTFB)
- new net: R?.1, R?.2, U?.12 (CAPFB)
- new net: Q?.4 (G), U?.15 (IGATE)
- new net: C?.1, U?.17 (CPF)
- new net: R?.1, R?.2, U?.19 (PFI)
- new net: R?.1, U?.2 (PROG)
- new net: L?.1, U?.21 (SW), U?.22 (SW)
- new net: JP?.1 (A), R?.2, U?.4 (~CHGEN)
- new net: JP?.1 (A), R?.2, U?.5 (~BSTEN)
- new net: Q?.1 (S), Q?.2 (S), Q?.3 (S), R?.1, U?.7 (CLN)
- new net +3.3V_BCKP: C?.1, C?.1, Q?.5 (D), R?.1, R?.1, R?.1, R?.1, R?.1, TP?.1 (TP), U?.1 (VSYS), U?.24 (VSYS)
- new net +3V3: C?.1, R?.1, R?.1, R?.1, R?.2, U?.16 (OVSNS), U?.6 (VIN)
- new net BCKP_CAPGD: R?.2, U?.13 (CAPGD)
- new net BCKP_IMON: U?.3 (IMON)
- new net BCKP_SYSGD: R?.2, U?.11 (SYSGD)
- new net GND: C?.2, C?.2, C?.2, C?.2, C?.2, JP?.2 (B), JP?.2 (B), R?.2, R?.2, R?.2, R?.2, U?.20 (CAPSEL), U?.25 (GND)
- new net VTANK: C?.1, L?.2, R?.1, TP?.1 (TP), U?.23 (SCAP)
- new net ~BCKP_CAPFLT: R?.2, U?.8 (~CAPFLT)
- new net ~BCKP_PFO: R?.2, U?.14 (~PFO)
- no-connect marks 0 -> 1
Other:
- note added: "Supercap Backup Circuit"
