File: hdw/Logic_Board/VFD_Clock/IO_Buffers.sch (KiCad schematic (older format))
At the start: 0 parts

Commit message: More work, project restructuring
Other:
- note removed: "Mechanical Components"
Changed lines of the file:
@@
 EELAYER 29 0
 EELAYER END
-$Descr A 11000 8500
+$Descr A4 11693 8268
 encoding utf-8
-Sheet 15 14
+Sheet 1 19
 Title ""
 Date ""
@@
 Comment4 ""
 $EndDescr
-Text Notes 4160 970  0    100  ~ 20
-Mechanical Components
 $EndSCHEMATC
