File: hdw/Display_Board/IV-8_Display_Board/Anode_Drivers.sch (KiCad schematic (older format))
At the start: 36 parts

Commit message: Added display board schematic, other additions to logic board
Parts:
- removed Q? (x6): BC856W, TO_SOT_Packages_SMD:SOT-323, symbol Transistor_BJT:BC856W
- removed Q? (x6): PMSTA06, TO_SOT_Packages_SMD:SOT-323, symbol Transistor_BJT:BC847W
- removed R? (x6): 10k, Resistors_SMD:R_0603, symbol Device:R
- removed R? (x6): 220k, Resistors_SMD:R_0603, symbol Device:R
- removed R? (x6): 68k, Resistors_SMD:R_0603, symbol Device:R
- removed R? (x6): 100k, Resistors_SMD:R_0603, symbol Device:R
- added Q? (x8): BC856W, TO_SOT_Packages_SMD:SOT-323, symbol Transistor_BJT:BC856W
- added Q? (x8): PMSTA06, TO_SOT_Packages_SMD:SOT-323, symbol Transistor_BJT:BC847W
- added R? (x8): 220k, Resistors_SMD:R_0603, symbol Device:R
- added R? (x8): 68k, Resistors_SMD:R_0603, symbol Device:R
- added R? (x8): 10k, Resistors_SMD:R_0603, symbol Device:R
- added R? (x8): 100k, Resistors_SMD:R_0603, symbol Device:R
Connections:
- net labels added: Anode_A, Anode_B, Anode_C, Anode_D, Anode_DP, Anode_E, Anode_F, Anode_G, drive_Anode_A, drive_Anode_B, drive_Anode_C, drive_Anode_D, drive_Anode_DP, drive_Anode_E, drive_Anode_F, drive_Anode_G
- net labels removed: Grid_0, Grid_1, Grid_2, Grid_3, Grid_4, Grid_5, VAN, drive_Grid_0, drive_Grid_1, drive_Grid_2, drive_Grid_3, drive_Grid_4, drive_Grid_5
- wire segments 48 -> 64
Other:
- note removed: "Grid Drivers"
