File: rev_b/hdw/Logic_Board/VFD_Clock/POS12_Telemetry.sch (KiCad schematic (older format))
At the start: 7 parts, among them U301 INA219BxDCN, U302 MCP9804

Commit message: PCB changes, deletions
Parts:
- U301, U302: Config (none) -> Telemetry
Changed lines of the file:
@@
 F 3 "http://ww1.microchip.com/downloads/en/DeviceDoc/22203b.pdf" H 4860 4990 50  0001 C CNN
 F 4 "MCP9804T-E/MCCT-ND" H 5110 4540 50  0001 C CNN "Digi-Key PN"
+F 5 "Telemetry" H 5110 4540 50  0001 C CNN "Config"
 	1    5110 4540
 	-1   0    0    -1
@@
 F 3 "http://www.ti.com/lit/ds/symlink/ina219.pdf" H 5460 1940 50  0001 C CNN
 F 4 "296-46420-1-ND" H 5110 2040 50  0001 C CNN "Digi-Key PN"
+F 5 "Telemetry" H 5110 2040 50  0001 C CNN "Config"
 	1    5110 2040
 	1    0    0    -1
