File: rev_b/hdw/Logic_Board/VFD_Clock/POS1P2_VFF_Telemetry.sch (KiCad schematic (older format))
At the start: 7 parts, among them U902 MCP9804, U903 INA219BxDCN

Commit message: PCB changes, deletions
Parts:
- U902, U903: Config (none) -> Telemetry
Changed lines of the file:
@@
 F 3 "http://ww1.microchip.com/downloads/en/DeviceDoc/22203b.pdf" H 5180 5290 50  0001 C CNN
 F 4 "MCP9804T-E/MCCT-ND" H 5430 4840 50  0001 C CNN "Digi-Key PN"
+F 5 "Telemetry" H 5430 4840 50  0001 C CNN "Config"
 	1    5430 4840
 	-1   0    0    -1
@@
 F 3 "http://www.ti.com/lit/ds/symlink/ina219.pdf" H 8560 2300 50  0001 C CNN
 F 4 "296-46420-1-ND" H 8210 2400 50  0001 C CNN "Digi-Key PN"
+F 5 "Telemetry" H 8210 2400 50  0001 C CNN "Config"
 	1    8210 2400
 	1    0    0    -1
