File: rev_b/hdw/Logic_Board/VFD_Clock/Time_of_Flight.sch (KiCad schematic (older format))
At the start: 7 parts, among them U2301 DS1683

Commit message: PCB changes, deletions
Parts:
- U2301: Config (none) -> TOF
Changed lines of the file:
@@
 F 3 "https://datasheets.maximintegrated.com/en/ds/DS1683.pdf" H 4740 4400 60  0001 C CNN
 F 4 "DS1683S+-ND" H 4940 3850 60  0001 C CNN "Digi-Key PN"
+F 5 "TOF" H 4840 4100 50  0001 C CNN "Config"
 	1    4840 4100
 	1    0    0    -1
