File: rev_b/hdw/Logic_Board/VFD_Clock/USB_Telemetry.sch (KiCad schematic (older format))
At the start: 7 parts, among them U2601 INA219BxDCN, U2602 MCP9804

Commit message: PCB changes, deletions
Parts:
- U2601, U2602: Config (none) -> Telemetry
Changed lines of the file:
@@
 F 3 "http://ww1.microchip.com/downloads/en/DeviceDoc/22203b.pdf" H 4860 4990 50  0001 C CNN
 F 4 "MCP9804T-E/MCCT-ND" H 5110 4540 50  0001 C CNN "Digi-Key PN"
+F 5 "Telemetry" H 5110 4540 50  0001 C CNN "Config"
 	1    5110 4540
 	-1   0    0    -1
@@
 F 3 "http://www.ti.com/lit/ds/symlink/ina219.pdf" H 5460 2000 50  0001 C CNN
 F 4 "296-46420-1-ND" H 5110 2100 50  0001 C CNN "Digi-Key PN"
+F 5 "Telemetry" H 5110 2100 50  0001 C CNN "Config"
 	1    5110 2100
 	1    0    0    -1
@@
 POS5_USB_SNS+
 $Comp
-L power:GND #PWR?
+L power:GND #PWR02609
 U 1 1 5F97036F
 P 5510 2300
-F 0 "#PWR?" H 5510 2050 50  0001 C CNN
+F 0 "#PWR02609" H 5510 2050 50  0001 C CNN
 F 1 "GND" V 5510 2150 50  0000 R CNN
 F 2 "" H 5510 2300 50  0001 C CNN
@@
 $EndComp
 $Comp
-L power:GND #PWR?
+L power:GND #PWR02610
 U 1 1 5F970A67
 P 5510 4640
-F 0 "#PWR?" H 5510 4390 50  0001 C CNN
+F 0 "#PWR02610" H 5510 4390 50  0001 C CNN
 F 1 "GND" V 5510 4490 50  0000 R CNN
 F 2 "" H 5510 4640 50  0001 C CNN
@@
 $EndComp
 $Comp
-L power:+3.3V #PWR?
+L power:+3.3V #PWR02611
 U 1 1 5F9716C3
 P 5510 4740
-F 0 "#PWR?" H 5510 4590 50  0001 C CNN
+F 0 "#PWR02611" H 5510 4590 50  0001 C CNN
 F 1 "+3.3V" V 5510 4880 50  0000 L CNN
 F 2 "" H 5510 4740 50  0001 C CNN
@@
 $EndComp
 $Comp
-L power:+3.3V #PWR?
+L power:+3.3V #PWR02612
 U 1 1 5F971BBA
 P 5510 4840
-F 0 "#PWR?" H 5510 4690 50  0001 C CNN
+F 0 "#PWR02612" H 5510 4690 50  0001 C CNN
 F 1 "+3.3V" V 5510 4980 50  0000 L CNN
 F 2 "" H 5510 4840 50  0001 C CNN
@@
 $EndComp
 $Comp
-L power:+3.3V #PWR?
+L power:+3.3V #PWR02601
 U 1 1 5F9742DA
 P 5110 1700
-F 0 "#PWR?" H 5110 1550 50  0001 C CNN
+F 0 "#PWR02601" H 5110 1550 50  0001 C CNN
 F 1 "+3.3V" H 5110 1840 50  0000 C CNN
 F 2 "" H 5110 1700 50  0001 C CNN
@@
 $EndComp
 $Comp
-L power:+3.3V #PWR?
+L power:+3.3V #PWR02603
 U 1 1 5F974784
 P 5110 2920
-F 0 "#PWR?" H 5110 2770 50  0001 C CNN
+F 0 "#PWR02603" H 5110 2770 50  0001 C CNN
 F 1 "+3.3V" H 5110 3060 50  0000 C CNN
 F 2 "" H 5110 2920 50  0001 C CNN
@@
 $EndComp
 $Comp
-L power:+3.3V #PWR?
+L power:+3.3V #PWR02605
 U 1 1 5F974D37
 P 5110 4040
-F 0 "#PWR?" H 5110 3890 50  0001 C CNN
+F 0 "#PWR02605" H 5110 3890 50  0001 C CNN
 F 1 "+3.3V" H 5110 4180 50  0000 C CNN
 F 2 "" H 5110 4040 50  0001 C CNN
@@
 $EndComp
 $Comp
-L power:+3.3V #PWR?
+L power:+3.3V #PWR02607
 U 1 1 5F9757DD
 P 5110 5540
-F 0 "#PWR?" H 5110 5390 50  0001 C CNN
+F 0 "#PWR02607" H 5110 5390 50  0001 C CNN
 F 1 "+3.3V" H 5110 5680 50  0000 C CNN
 F 2 "" H 5110 5540 50  0001 C CNN
@@
 $EndComp
 $Comp
-L power:GND #PWR?
+L power:GND #PWR02602
 U 1 1 5F977F14
 P 5110 2500
-F 0 "#PWR?" H 5110 2250 50  0001 C CNN
+F 0 "#PWR02602" H 5110 2250 50  0001 C CNN
 F 1 "GND" H 5110 2350 50  0000 C CNN
 F 2 "" H 5110 2500 50  0001 C CNN
@@
 $EndComp
 $Comp
-L power:GND #PWR?
+L power:GND #PWR02604
 U 1 1 5F978327
 P 5110 3220
-F 0 "#PWR?" H 5110 2970 50  0001 C CNN
+F 0 "#PWR02604" H 5110 2970 50  0001 C CNN
 F 1 "GND" H 5110 3070 50  0000 C CNN
 F 2 "" H 5110 3220 50  0001 C CNN
@@
 $EndComp
 $Comp
-L power:GND #PWR?
+L power:GND #PWR02606
 U 1 1 5F9786FB
 P 5110 5120
-F 0 "#PWR?" H 5110 4870 50  0001 C CNN
+F 0 "#PWR02606" H 5110 4870 50  0001 C CNN
 F 1 "GND" H 5110 4970 50  0000 C CNN
 F 2 "" H 5110 5120 50  0001 C CNN
@@
 $EndComp
 $Comp
-L power:GND #PWR?
+L power:GND #PWR02608
 U 1 1 5F978E58
 P 5110 5840
-F 0 "#PWR?" H 5110 5590 50  0001 C CNN
+F 0 "#PWR02608" H 5110 5590 50  0001 C CNN
 F 1 "GND" H 5110 5690 50  0000 C CNN
 F 2 "" H 5110 5840 50  0001 C CNN
