File: rev_b/hdw/Logic_Board/VFD_Clock/Microcontroller_Clocking.sch (KiCad schematic (older format))
At the start: 13 parts, among them X1701 ASE-8.000MHz, X1702 ECS-327KE

Commit message: More sch work, ran ERC
Connections:
- net +3.3V_BCKP renamed +3V3
Changed lines of the file:
@@
 	5510 1800 6400 1800
 Connection ~ 5510 1800
-$Comp
-L Custom_Library:+3.3V_BCKP #PWR01701
-U 1 1 5E054361
-P 4530 1720
-F 0 "#PWR01701" H 4530 1570 50  0001 C CNN
-F 1 "+3.3V_BCKP" H 4530 1860 50  0000 C CNN
-F 2 "" H 4530 1720 50  0000 C CNN
-F 3 "" H 4530 1720 50  0000 C CNN
-	1    4530 1720
-	1    0    0    -1
-$EndComp
 Wire Wire Line
 	4530 1720 4530 1800
@@
 	5510 4290 6400 4290
 Connection ~ 5510 4290
-$Comp
-L Custom_Library:+3.3V_BCKP #PWR01702
-U 1 1 5E05633B
-P 4530 4210
-F 0 "#PWR01702" H 4530 4060 50  0001 C CNN
-F 1 "+3.3V_BCKP" H 4530 4350 50  0000 C CNN
-F 2 "" H 4530 4210 50  0000 C CNN
-F 3 "" H 4530 4210 50  0000 C CNN
-	1    4530 4210
-	1    0    0    -1
-$EndComp
 Wire Wire Line
 	4530 4210 4530 4290
@@
 Wire Wire Line
 	6400 4330 6720 4330
+$Comp
+L power:+3.3V #PWR0101
+U 1 1 5F87C21E
+P 4530 4210
+F 0 "#PWR0101" H 4530 4060 50  0001 C CNN
+F 1 "+3.3V" H 4530 4350 50  0000 C CNN
+F 2 "" H 4530 4210 50  0001 C CNN
+F 3 "" H 4530 4210 50  0001 C CNN
+	1    4530 4210
+	1    0    0    -1
+$EndComp
+$Comp
+L power:+3.3V #PWR0102
+U 1 1 5F87CA12
+P 4530 1720
+F 0 "#PWR0102" H 4530 1570 50  0001 C CNN
+F 1 "+3.3V" H 4530 1860 50  0000 C CNN
+F 2 "" H 4530 1720 50  0001 C CNN
+F 3 "" H 4530 1720 50  0001 C CNN
+	1    4530 1720
+	1    0    0    -1
+$EndComp
 $EndSCHEMATC
